File: Schematics/Z80-GPU/Z80-GPU.kicad_sch (KiCad schematic)
At the start: 63 parts

Commit message: New features
Parts:
- J?: value (none) -> Conn_02x04_Odd_Even
- U?: value (none) -> 74F86
- U?: value (none) -> 74LS02
- U?: value (none) -> 74F00
- U?: value (none) -> 74LS163
- U?: value (none) -> 74LS13
- U?: value (none) -> 74HCT157
- U?: value (none) -> 74LS06
- U?: value (none) -> 74LS174
- U?: value (none) -> 74HCT166
- U?: value (none) -> 74LS245
- U?: value (none) -> 74LS32
- U?: value (none) -> 74LS74
Other:
- moved on the sheet: U?
