File: Schematics/Z80-MIDI/z80-MIDI.kicad_sch (KiCad schematic)
At the start: 37 parts, among them J1 Conn_02x32_Row_Letter_First, J3 DB9_Male, J6 DIN-5, J7 DIN-5, U14 74LS06, U18 6N137, U19 74LS06, U20 74LS02, X1 1MHz

Commit message: New features
Parts:
- IC1: value (none) -> SIO0-DIP-40; footprint (none) -> Package_DIP:DIP-40_W15.24mm_Socket_LongPads
- J2: value (none) -> Conn_02x05_Odd_Even; footprint (none) -> Connector_PinHeader_2.54mm:PinHeader_2x05_P2.54mm_Vertical
- J4: value (none) -> DB9_Male
- J5: value (none) -> Conn_02x04_Odd_Even; footprint (none) -> Connector_PinHeader_2.54mm:PinHeader_2x04_P2.54mm_Vertical
- U1: value (none) -> 74LS688; footprint (none) -> Package_DIP:DIP-20_W7.62mm_Socket_LongPads
- U10: footprint (none) -> Package_DIP:DIP-16_W7.62mm_Socket_LongPads
- U11: value (none) -> 74HCT4051; footprint (none) -> Package_DIP:DIP-16_W7.62mm_Socket_LongPads
- U12: value (none) -> AD570; footprint (none) -> Package_DIP:DIP-18_W7.62mm_Socket_LongPads
- U13, U2, U3, U4: value (none) -> 74HC245; footprint (none) -> Package_DIP:DIP-20_W7.62mm_Socket_LongPads
- U14: value 74LS06 -> (none); footprint Package_DIP:DIP-14_W7.62mm_Socket_LongPads -> (none)
- U14: value 74LS06 -> (none)
- U15: value (none) -> LM7915_TO220; footprint (none) -> Package_TO_SOT_THT:TO-220-3_Vertical
- U16: value (none) -> LM7810_TO220; footprint (none) -> Package_TO_SOT_THT:TO-220-3_Vertical
- U17: value (none) -> LM7910_TO220; footprint (none) -> Package_TO_SOT_THT:TO-220-3_Vertical
- U5: value (none) -> 74HC02; footprint (none) -> Package_DIP:DIP-14_W7.62mm_Socket_LongPads
- U6: value (none) -> 74HC138; footprint (none) -> Package_DIP:DIP-16_W7.62mm_Socket_LongPads
- U7, U8, U9: value (none) -> 74LS573; footprint (none) -> Package_DIP:DIP-20_W7.62mm_Socket_LongPads
