File: Schematics/Z80-IDE/Z80-IDE.kicad_sch (KiCad schematic)
At the start: 65 parts, among them CON1 CF-CARD, J1 Conn_02x32_Row_Letter_First, J2 IDE Connector, J3 Floppy Connector, Q1 BC548, U1 74HC74, U10 74HCT04, U11 74HC14, U12 74HCT139, U13 FDC9266, U15 L7805, U16 74HCT04, U17 74HC240, U2 74LS688, U3 74HC245, U4 74HC245, U5 74HC245, U6 74HC02, U7 82C55A_PLCC, U8 GAL16V8, U9 74HCT273, X1 8MHz

Commit message: Updated
Parts:
- U11: value 74HC14 -> 74HCT14
