File: Schematics/Z80-IDE/Z80-IDE.kicad_pcb (KiCad board)
At the start: 2 copper layers, 160 x 100.3 mm, 62 parts, among them CON1 CF-CARD, J1 Conn_02x32_Row_Letter_First, J2 IDE Connector, J3 Floppy Connector, Q1 BC548, U1 74HC74, U10 74HCT04, U11 74HC14, U12 74HCT139, U13 FDC9266, U15 L7805, U16 74HCT04, U17 74HC240, U2 74LS688, U3 74HC245, U4 74HC245, U5 74HC245, U6 74HC02, U7 82C55A_PLCC, U8 GAL16V8, U9 74HCT273, X1 8MHz

Commit message: added i2c controller functions, added IDE interface functions, fiexd IDE schematics
Parts:
- U11: value 74HC14 -> 74HCT14
Connections:
- U8 pad 8: unconnected-(U8-Pad8) -> /~{#RD}
Changed lines of the file:
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@@
   (net 216 "unconnected-(U8-Pad6)")
   (net 217 "unconnected-(U8-Pad7)")
-  (net 218 "unconnected-(U8-Pad8)")
   (footprint "Resistor_THT:R_Axial_DIN0204_L3.6mm_D1.6mm_P2.54mm_Vertical" (layer "F.Cu")
     (at 214.63 134.62)
@@
       (effects (font (size 1 1) (thickness 0.15)))
     )
-    (fp_text value "74HC14" (at 3.81 17.57) (layer "F.Fab")
+    (fp_text value "74HCT14" (at 3.81 17.57) (layer "F.Fab")
       (effects (font (size 1 1) (thickness 0.15)))
     )
@@
       (net 217 "unconnected-(U8-Pad7)") (pinfunction "I7") (pintype "input"))
     (pad "8" thru_hole oval (at 0 17.78) (size 2.4 1.6) (drill 0.8) (layers *.Cu *.Mask)
-      (net 218 "unconnected-(U8-Pad8)") (pinfunction "I8") (pintype "input"))
+      (net 115 "/~{#RD}") (pinfunction "I8") (pintype "input"))
     (pad "9" thru_hole oval (at 0 20.32) (size 2.4 1.6) (drill 0.8) (layers *.Cu *.Mask)
       (net 129 "/~{#IOREQ}") (pinfunction "I9") (pintype "input"))
