File: Schematics/Z80-MIO/Z80-MIO.kicad_pcb (KiCad board)
At the start: 2 copper layers, 160 x 100.3 mm, 77 parts, among them J1 Conn_02x05_Odd_Even, J2 Conn_02x32_Row_Letter_First, J3 Conn_02x02_Top_Bottom, J4 Conn_02x06_Odd_Even, J5 Mini-DIN-6, J6 Mini-DIN-6, J7 Jumper_2_Bridged, J8 Conn_02x04_Odd_Even, J9 Conn_02x04_Odd_Even, Q1 BC548, U1 74HC688, U10 DS1307+, U11 74HC161, U12 Am9511A, U2 GAL16V8, U3 74HC245, U4 74HC245, U5 74HC245, U6 PIO-DIP-40, U7 74LS06, U8 PCF8584, U9 8048, Y1 32.768 kHz

Commit message: Updated
Connections:
- U1 pad 2: //IOREQ -> /~{#IOREQ}
- U1 pad 4: //IOREQ -> /~{#IOREQ}
- U1 pad 6: //IOREQ -> /~{#IOREQ}
- U1 pad 8: //IOREQ -> /~{#IOREQ}
Routing:
- net /~{#IOREQ}: track 114.2 -> 173.3 mm, vias 2 -> 3
- net //IOREQ: track 18.9 -> 0.00 mm
- net KBCI: track 50.6 -> 57.4 mm, vias 1 -> 2
- net MSCI: track 45.1 -> 50.0 mm, vias 0 -> 1
- net GND: track 1118.0 -> 1114.8 mm
- net KBDI: track 93.2 -> 94.9 mm, vias 1 -> 2
- net MSDI: track 82.2 -> 83.3 mm
- net +5V: track 810.7 -> 811.7 mm
Other:
- board text added: "J3 I2C Routing 1-2 SDA>A23 3-4 SDC>A22"
- board text added: "J8 APU Int 1-2 INT0 3-4 INT1 5-6 INT2 7-8 INT3"
- board text added: "J9 APU Clock 1-2 /2 3-4 /4 5-6 /8 7-8 /16 Max. 3MHz"
- board text added: "Z8C Multi I/O Board Rev.2 2022 - www.dennisgunia.de"
- board text removed: "J2 I2C Routing 1-2 SDA>A23 3-4 SDC>A22"
- board text removed: "J7 APU Int 1-2 INT0 3-4 INT1 5-6 INT2 7-8 INT3"
- board text removed: "J8 APU Clock 1-2 /2 3-4 /4 5-6 /8 7-8 /16 Max. 3MHz"
- board text removed: "Z8C Multi I/O Board 2022 - www.dennisgunia.de"
