File: Schematics/Z80-MIO/Z80-MIO.kicad_sch (KiCad schematic)
At the start: 77 parts, among them J1 Conn_02x05_Odd_Even, J2 Conn_02x32_Row_Letter_First, J3 Conn_02x02_Top_Bottom, J4 Conn_02x06_Odd_Even, J5 Mini-DIN-6, J6 Mini-DIN-6, J7 Jumper_2_Bridged, J8 Conn_02x04_Odd_Even, J9 Conn_02x04_Odd_Even, Q1 BC548, U1 74HC688, U10 DS1307+, U11 74HC161, U12 Am9511A, U2 GAL16V8, U3 74HC245, U4 74HC245, U5 74HC245, U6 PIO-DIP-40, U7 74LS06, U8 PCF8584, U9 8048, Y1 32.768 kHz

Commit message: Updated
Parts:
- U3: value 74HC245 -> 74HC2T45
- U7: value 74LS06 -> 7406
Connections:
- net /IOREQ is gone; now on net ~{#IOREQ}: U1.2 (P0), U1.4 (P1), U1.6 (P2), U1.8 (P3)
Changed lines of the file:
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@@
     (title "Z8C MIO Board")
     (date "2022-10-10")
+    (rev "2")
     (comment 1 "Multi I/O Board for Z8C")
     (comment 2 "Interrupt-Controller, GPIO, PS2, I2C, RTC, FPU/APU and Speaker")
@@
     (effects (font (size 1.27 1.27)) (justify right bottom))
   )
-  (label "/IOREQ" (at 47.371 29.337 0)
+  (label "~{#IOREQ}" (at 47.371 29.337 0)
     (effects (font (size 1.27 1.27)) (justify left bottom))
   )
@@
     (in_bom yes) (on_board yes)
     (property "Reference" "U7" (id 0) (at 267.081 39.7002 0))
-    (property "Value" "74LS06" (id 1) (at 267.081 42.0116 0))
+    (property "Value" "7406" (id 1) (at 267.081 42.0116 0))
     (property "Footprint" "Package_DIP:DIP-14_W7.62mm_Socket" (id 2) (at 267.081 47.752 0)
       (effects (font (size 1.27 1.27)) hide)
@@
     (pin "1")
     (pin "2")
-    (pin "3")
-    (pin "4")
-    (pin "5")
-    (pin "6")
-    (pin "8")
-    (pin "9")
-    (pin "10")
-    (pin "11")
-    (pin "12")
-    (pin "13")
-    (pin "14")
-    (pin "7")
   )
   (symbol (lib_id "Connector_Generic:Conn_02x05_Odd_Even") (at 40.386 83.312 90) (unit 1)
@@
     (in_bom yes) (on_board yes)
     (property "Reference" "U7" (id 0) (at 148.971 60.6552 0))
-    (property "Value" "74LS06" (id 1) (at 148.971 62.9666 0))
+    (property "Value" "7406" (id 1) (at 148.971 62.9666 0))
     (property "Footprint" "Package_DIP:DIP-14_W7.62mm_Socket" (id 2) (at 148.971 68.707 0)
       (effects (font (size 1.27 1.27)) hide)
@@
       (effects (font (size 1.27 1.27)) hide)
     )
-    (pin "1")
-    (pin "2")
-    (pin "3")
-    (pin "4")
-    (pin "5")
-    (pin "6")
-    (pin "8")
-    (pin "9")
     (pin "10")
     (pin "11")
-    (pin "12")
-    (pin "13")
-    (pin "14")
-    (pin "7")
   )
   (symbol (lib_id "Device:R_Network08") (at 24.511 59.817 90) (unit 1)
@@
     (in_bom yes) (on_board yes)
     (property "Reference" "U7" (id 0) (at 267.081 91.7702 0))
-    (property "Value" "74LS06" (id 1) (at 267.081 94.0816 0))
+    (property "Value" "7406" (id 1) (at 267.081 94.0816 0))
     (property "Footprint" "Package_DIP:DIP-14_W7.62mm_Socket" (id 2) (at 267.081 99.822 0)
       (effects (font (size 1.27 1.27)) hide)
@@
       (effects (font (size 1.27 1.27)) hide)
     )
-    (pin "1")
-    (pin "2")
-    (pin "3")
-    (pin "4")
-    (pin "5")
-    (pin "6")
     (pin "8")
     (pin "9")
-    (pin "10")
-    (pin "11")
-    (pin "12")
-    (pin "13")
-    (pin "14")
-    (pin "7")
   )
   (symbol (lib_id "power:GND") (at 82.296 177.292 0) (unit 1)
     (in_bom yes) (on_board yes) (fields_autoplaced)
-    (property "Reference" "#PWR?" (id 0) (at 82.296 183.642 0)
+    (property "Reference" "#PWR0101" (id 0) (at 82.296 183.642 0)
       (effects (font (size 1.27 1.27)) hide)
     )
@@
     (in_bom yes) (on_board yes)
     (property "Reference" "U7" (id 0) (at 267.081 70.1802 0))
-    (property "Value" "74LS06" (id 1) (at 267.081 72.4916 0))
+    (property "Value" "7406" (id 1) (at 267.081 72.4916 0))
     (property "Footprint" "Package_DIP:DIP-14_W7.62mm_Socket" (id 2) (at 267.081 78.232 0)
       (effects (font (size 1.27 1.27)) hide)
@@
       (effects (font (size 1.27 1.27)) hide)
     )
-    (pin "1")
-    (pin "2")
-    (pin "3")
-    (pin "4")
     (pin "5")
     (pin "6")
-    (pin "8")
-    (pin "9")
-    (pin "10")
-    (pin "11")
-    (pin "12")
-    (pin "13")
-    (pin "14")
-    (pin "7")
   )
   (symbol (lib_id "power:+5V") (at 208.026 191.262 0) (unit 1)
@@
       (effects (font (size 1.27 1.27)) (justify left))
     )
-    (property "Value" "74LS06" (id 1) (at 281.813 153.67 0)
+    (property "Value" "7406" (id 1) (at 281.813 153.67 0)
       (effects (font (size 1.27 1.27)) (justify left))
     )
@@
       (effects (font (size 1.27 1.27)) hide)
     )
-    (pin "1")
-    (pin "2")
-    (pin "3")
-    (pin "4")
-    (pin "5")
-    (pin "6")
-    (pin "8")
-    (pin "9")
-    (pin "10")
-    (pin "11")
-    (pin "12")
-    (pin "13")
     (pin "14")
     (pin "7")
@@
     (in_bom yes) (on_board yes)
     (property "Reference" "U7" (id 0) (at 267.081 18.1102 0))
-    (property "Value" "74LS06" (id 1) (at 267.081 20.4216 0))
+    (property "Value" "7406" (id 1) (at 267.081 20.4216 0))
     (property "Footprint" "Package_DIP:DIP-14_W7.62mm_Socket" (id 2) (at 267.081 26.162 0)
       (effects (font (size 1.27 1.27)) hide)
@@
       (effects (font (size 1.27 1.27)) hide)
     )
-    (pin "1")
-    (pin "2")
     (pin "3")
     (pin "4")
-    (pin "5")
-    (pin "6")
-    (pin "8")
-    (pin "9")
-    (pin "10")
-    (pin "11")
-    (pin "12")
-    (pin "13")
-    (pin "14")
-    (pin "7")
   )
   (symbol (lib_id "power:+5V") (at 295.021 37.592 0) (unit 1)
@@
     (in_bom yes) (on_board yes)
     (property "Reference" "U7" (id 0) (at 148.971 75.8952 0))
-    (property "Value" "74LS06" (id 1) (at 148.971 78.2066 0))
+    (property "Value" "7406" (id 1) (at 148.971 78.2066 0))
     (property "Footprint" "Package_DIP:DIP-14_W7.62mm_Socket" (id 2) (at 148.971 83.947 0)
       (effects (font (size 1.27 1.27)) hide)
@@
       (effects (font (size 1.27 1.27)) hide)
     )
-    (pin "1")
-    (pin "2")
-    (pin "3")
-    (pin "4")
-    (pin "5")
-    (pin "6")
-    (pin "8")
-    (pin "9")
-    (pin "10")
-    (pin "11")
     (pin "12")
     (pin "13")
-    (pin "14")
-    (pin "7")
   )
   (symbol (lib_id "power:+12V") (at 378.206 29.972 0) (unit 1)
@@
   (symbol (lib_id "74xx:74HC245") (at 94.996 164.592 0) (unit 1)
     (in_bom yes) (on_board yes) (fields_autoplaced)
-    (property "Reference" "U3" (id 0) (at 97.0154 143.637 0)
+    (property "Reference" "U3" (id 0) (at 97.0154 143.51 0)
       (effects (font (size 1.27 1.27)) (justify left))
     )
-    (property "Value" "74HC245" (id 1) (at 97.0154 146.177 0)
+    (property "Value" "74HC2T45" (id 1) (at 97.0154 146.05 0)
       (effects (font (size 1.27 1.27)) (justify left))
     )
-    (property "Footprint" "Package_DIP:DIP-20_W7.62mm_LongPads" (id 2) (at 94.996 164.592 0))
+    (property "Footprint" "Package_DIP:DIP-20_W7.62mm_LongPads" (id 2) (at 94.996 164.592 0)
+      (effects (font (size 1.27 1.27)) hide)
+    )
     (property "Datasheet" "http://www.ti.com/lit/gpn/sn74HC245" (id 3) (at 94.996 164.592 0)
       (effects (font (size 1.27 1.27)) hide)
@@
     )
     (path "/45ab63b2-69a7-4901-a31d-21ac38882192"
-      (reference "#PWR?") (unit 1) (value "GND") (footprint "")
+      (reference "#PWR0101") (unit 1) (value "GND") (footprint "")
     )
     (path "/8e7180ee-df11-413a-a15b-c8e45c120046"
@@
     )
     (path "/d2e530a1-503a-40ca-b72f-2bf31ec0fb32"
-      (reference "U3") (unit 1) (value "74HC245") (footprint "Package_DIP:DIP-20_W7.62mm_LongPads")
+      (reference "U3") (unit 1) (value "74HC2T45") (footprint "Package_DIP:DIP-20_W7.62mm_LongPads")
     )
     (path "/44d50cf2-8bea-4112-9d30-477d02e50476"
@@
     )
     (path "/2ddc9543-f16e-46ae-8d39-b2918a5be067"
-      (reference "U7") (unit 1) (value "74LS06") (footprint "Package_DIP:DIP-14_W7.62mm_Socket")
+      (reference "U7") (unit 1) (value "7406") (footprint "Package_DIP:DIP-14_W7.62mm_Socket")
     )
     (path "/7e042812-9033-4877-9152-b031dd83a033"
-      (reference "U7") (unit 2) (value "74LS06") (footprint "Package_DIP:DIP-14_W7.62mm_Socket")
+      (reference "U7") (unit 2) (value "7406") (footprint "Package_DIP:DIP-14_W7.62mm_Socket")
     )
     (path "/63358355-bbc3-4796-abc2-498c9d08668f"
-      (reference "U7") (unit 3) (value "74LS06") (footprint "Package_DIP:DIP-14_W7.62mm_Socket")
+      (reference "U7") (unit 3) (value "7406") (footprint "Package_DIP:DIP-14_W7.62mm_Socket")
     )
     (path "/4572e6a2-b528-408d-9ec4-54ae9300ab05"
-      (reference "U7") (unit 4) (value "74LS06") (footprint "Package_DIP:DIP-14_W7.62mm_Socket")
+      (reference "U7") (unit 4) (value "7406") (footprint "Package_DIP:DIP-14_W7.62mm_Socket")
     )
     (path "/41c1dbec-e911-4a87-9b07-0f0166125df9"
-      (reference "U7") (unit 5) (value "74LS06") (footprint "Package_DIP:DIP-14_W7.62mm_Socket")
+      (reference "U7") (unit 5) (value "7406") (footprint "Package_DIP:DIP-14_W7.62mm_Socket")
     )
     (path "/cf1c44d8-562d-4508-a840-78f4aed0f2ee"
-      (reference "U7") (unit 6) (value "74LS06") (footprint "Package_DIP:DIP-14_W7.62mm_Socket")
+      (reference "U7") (unit 6) (value "7406") (footprint "Package_DIP:DIP-14_W7.62mm_Socket")
     )
     (path "/7bf15ebd-56f9-4728-9fb7-e8f3a6246770"
-      (reference "U7") (unit 7) (value "74LS06") (footprint "Package_DIP:DIP-14_W7.62mm_Socket")
+      (reference "U7") (unit 7) (value "7406") (footprint "Package_DIP:DIP-14_W7.62mm_Socket")
     )
     (path "/b235e860-eb06-4b98-9bc2-972f8490f3de"
