File: Schematics/Z80-X86CPU/Z80-X86CPU.kicad_sch (KiCad schematic)
At the start: 10 parts

Commit message: added i2c controller tests
Parts:
- added C? (x2): 100nF, Capacitor_THT:C_Rect_L7.0mm_W2.0mm_P5.00mm, symbol Device:C_Small
- added R?: 4.7k, Resistor_THT:R_Axial_DIN0204_L3.6mm_D1.6mm_P2.54mm_Vertical, symbol Device:R
- added SW?: SW_SPDT, digikey-footprints:Toggle_Switch_100SP1T2B4M6QE, symbol Switch:SW_SPDT
- added U? (x2): IS61C5128AS-25QLI, Package_SO:SSOP-32_11.305x20.495mm_P1.27mm, symbol Memory_RAM:IS61C5128AS-25QLI
- added U?: 74LS04, symbol 74xx:74LS04
- added U? (x3): 74LS157, symbol 74xx:74LS157
- added Y?: 24MHz, symbol Device:Crystal
- R?: value (none) -> 4.7K
- U?: value (none) -> 8088; footprint (none) -> Package_DIP:DIP-40_W15.24mm
- U?: value (none) -> 8259; footprint (none) -> Package_DIP:DIP-28_W15.24mm
- U?: value (none) -> 74LS245
- U?: value (none) -> 8284; footprint (none) -> Package_DIP:DIP-18_W7.62mm
- U?: value (none) -> 8288; footprint (none) -> Package_DIP:DIP-20_W7.62mm
- U?: value (none) -> 74LS00
- U?: value (none) -> 74HCT573
Connections:
- net +5V: now also U?.31 (HOLD), U?.7 (~{AEN2}), C?.1, R?.1, U?.32 (VDD), U?.32 (VDD)
- net CPU_A0: now also U?.12 (A0), U?.12 (A0), U?.2 (I0a)
- net CPU_A1: now also U?.11 (A1), U?.11 (A1), U?.5 (I0b)
- net CPU_A10: now also U?.23 (A10), U?.23 (A10), U?.3 (I1a)
- net CPU_A11: now also U?.25 (A11), U?.25 (A11), U?.6 (I1b)
- net CPU_A12: now also U?.10 (I1c), U?.4 (A12), U?.4 (A12)
- net CPU_A13: now also U?.13 (I1d), U?.28 (A13), U?.28 (A13)
- net CPU_A14: now also U?.3 (A14), U?.3 (A14), U?.3 (I1a)
- net CPU_A15: now also U?.31 (A15), U?.31 (A15), U?.6 (I1b)
- net CPU_A16: now also U?.10 (I1c), U?.2 (A16), U?.2 (A16)
- net CPU_A17: now also U?.1 (A17), U?.1 (A17), U?.13 (I1d)
- net CPU_A18: now also U?.3 (I1a), U?.30 (A18), U?.30 (A18)
- net CPU_A19: now also U?.1, U?.22 (~{CE}), U?.6 (I1b)
- net CPU_A2: now also U?.10 (A2), U?.10 (A2), U?.11 (I0c)
- net CPU_A3: now also U?.14 (I0d), U?.9 (A3), U?.9 (A3)
- net CPU_A4: now also U?.2 (I0a), U?.8 (A4), U?.8 (A4)
- net CPU_A5: now also U?.5 (I0b), U?.7 (A5), U?.7 (A5)
- net CPU_A6: now also U?.11 (I0c), U?.6 (A6), U?.6 (A6)
- net CPU_A7: now also U?.14 (I0d), U?.5 (A7), U?.5 (A7)
- net CPU_A8: now also U?.2 (I0a), U?.27 (A8), U?.27 (A8)
- net CPU_A9: now also U?.26 (A9), U?.26 (A9), U?.5 (I0b)
- net CPU_CLK: now also U?.8 (CLK)
- net CPU_D0: now also U?.13 (I/O0), U?.13 (I/O0)
- net CPU_D1: now also U?.14 (I/O1), U?.14 (I/O1)
- net CPU_D2: now also U?.15 (I/O2), U?.15 (I/O2)
- net CPU_D3: now also U?.17 (I/O3), U?.17 (I/O3)
- net CPU_D4: now also U?.18 (I/O4), U?.18 (I/O4)
- net CPU_D5: now also U?.19 (I/O5), U?.19 (I/O5)
- net CPU_D6: now also U?.20 (I/O6), U?.20 (I/O6)
- net CPU_D7: now also U?.21 (I/O7), U?.21 (I/O7)
- net GND: now also U?.1 (CSYNC), U?.13 (F/~{C}), U?.15 (~{ASYNC}), U?.33 (MN/~{MX}), U?.6 (RDY2), C?.2, SW?.2 (B), U?.16 (GND), U?.16 (GND)
- net CPU_RESET: now reaches U?.21 (RESET)
- net CPU_RESET: now also U?.10 (RESET)
- net CPU_READY: now reaches U?.22 (READY)
- net CPU_READY: now also U?.5 (READY)
- net at U?.11 (~{RES}): now also C?.2, R?.2, SW?.3 (C)
- net CPU_OSC: now reaches U?.12 (OSC)
- net at U?.16 (X2): now also Y?.2
- net at U?.17 (X1): now also C?.1, Y?.1
- net CPU_PCLK: now reaches U?.2 (PCLK)
- net CPU_~{MRDC}: now reaches U?.7 (~{MRDC})
- net CPU_~{MRDC}: now also U?.24 (~{OE}), U?.24 (~{OE})
- net CPU_~{MWTC}: now reaches U?.9 (~{MWTC})
- net CPU_~{MWTC}: now also U?.29 (~{WE}), U?.29 (~{WE})
- new net ~{CPU_A19}: U?.2, U?.22 (~{CE})
- no-connect marks 3 -> 7
Other:
- note added: "RESET"
- moved on the sheet: R?, U?, U?A
