File: Modules/001-CPU Board V1/Schematics/Z80.kicad_sch (KiCad schematic)
At the start: 65 parts, among them J1 CTC_CLK_SEL, J2 CON_FTDI, J3 ROM_/WR_EN, J4 DB9_Female, J5 Barrel_Jack, J6 Conn_02x32_Row_Letter_First, Q1 BC548, Q2 BC548, SW1 SW_DIP_x08, SW2 SW_SPDT, U1 Z80CPU, U10 NE555P, U11 GAL16V8, U12 74HC245, U13 CTC-DIP-28, U14 SIO0-DIP-40, U15 MAX232, U2 HM62256BLP, U3 HM62256BLP, U4 28C256, U5 74HC137, U6 74HC00, U7 74HC02, U8 74HC74, U9 74HC14, X1 3.686411MHz, X2 7.372800MHz

Commit message: multiple updates
Other:
- note added: "POSSIBLE MOD: - disconnect U7 Pin 13 - bridge U7 Pin 12+13 - disconnect U5 Pin 6 - connect MEMAQ to U5 Pin 6 => MEMAQ now works in the full 64k range"
Changed lines of the file:
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@@
     (stroke (width 0) (type default))
   )
-  (wire (pts (xy 92.71 91.44) (xy 92.71 96.52))
+  (wire (pts (xy 92.71 91.44) (xy 92.71 95.25))
     (stroke (width 0) (type default))
   )
@@
     (effects (font (size 1.27 1.27)) (justify left bottom))
   )
+  (text "POSSIBLE MOD:\n- disconnect U7 Pin 13\n- bridge U7 Pin 12+13\n- disconnect U5 Pin 6\n- connect MEMAQ to U5 Pin 6\n=> MEMAQ now works in the full 64k range"
+    (at 72.39 109.22 0)
+    (effects (font (size 1.27 1.27)) (justify left bottom))
+  )
   (text "$0000-3FFF\n" (at 198.755 18.415 0)
     (effects (font (size 1.27 1.27)) (justify right bottom))
@@
     )
   )
-  (symbol (lib_id "power:GND") (at 92.71 96.52 0) (unit 1)
-    (in_bom yes) (on_board yes) (dnp no) (fields_autoplaced)
-    (property "Reference" "#PWR0103" (at 92.71 102.87 0)
+  (symbol (lib_id "power:GND") (at 92.71 95.25 0) (unit 1)
+    (in_bom yes) (on_board yes) (dnp no)
+    (property "Reference" "#PWR0103" (at 92.71 101.6 0)
       (effects (font (size 1.27 1.27)) hide)
     )
-    (property "Value" "GND" (at 92.71 101.6 0)
+    (property "Value" "GND" (at 96.52 96.52 0)
       (effects (font (size 1.27 1.27)))
     )
-    (property "Footprint" "" (at 92.71 96.52 0)
+    (property "Footprint" "" (at 92.71 95.25 0)
       (effects (font (size 1.27 1.27)) hide)
     )
-    (property "Datasheet" "" (at 92.71 96.52 0)
+    (property "Datasheet" "" (at 92.71 95.25 0)
       (effects (font (size 1.27 1.27)) hide)
     )
