File: Modules/XXX-Future Ideas/Z80-MIDI/z80-MIDI.kicad_sch (KiCad schematic)
At the start: 37 parts, among them IC1 SIO0-DIP-40, J1 Conn_02x32_Row_Letter_First, J2 Conn_02x05_Odd_Even, J3 DB9_Male, J4 DB9_Male, J5 Conn_02x04_Odd_Even, J6 DIN-5, J7 DIN-5, U1 74LS688, U11 74HCT4051, U12 AD570, U13 74HC245, U15 LM7915_TO220, U16 LM7810_TO220, U17 LM7910_TO220, U18 6N137, U19 74LS06, U2 74HC245, U20 74LS02, U3 74HC245, U4 74HC245, U5 74HC02, U6 74HC138, U7 74LS573, U8 74LS573, U9 74LS573, X1 1MHz

Commit message: multiple updates
Parts:
- removed J1: Conn_02x32_Row_Letter_First, Connector_DIN:DIN41612_Q_2x32_Male_Horizontal_THT, symbol Connector_Generic:Conn_02x32_Row_Letter_First
- removed unit 2 of U5
- removed unit 3 of U5
- removed U7, U9: 74LS573, Package_DIP:DIP-20_W7.62mm_Socket_LongPads, symbol 74xx:74LS573
- added J8: Z8C_Card, Dennis:Z8C Card, symbol Dennis:Z8C_Card
- added U21: PIO-DIP-40, Package_DIP:DIP-40_W15.24mm_Socket, symbol Zilog_Z80_Peripherals:PIO-DIP-40
- IC1: footprint Package_DIP:DIP-40_W15.24mm_Socket_LongPads -> Package_DIP:DIP-40_W15.24mm_Socket
- J3, J4: footprint (none) -> Connector_Dsub:DSUB-9_Female_Horizontal_P2.77x2.84mm_EdgePinOffset4.94mm_Housed_MountingHolesOffset7.48mm
- U10: value (none) -> 74HC590
- U14: value (none) -> 74HCT04
Connections:
- net ~{RD_PORTA} is gone; now on net ~{CS_SIO}: U6.15 (O0)
- net #A0: now also U21.5 (C/~{D}); no longer U6.1 (A0)
- net #A1: now also U21.6 (B/~{A}); no longer U6.2 (A1)
- net #A2: now also U6.1 (A0); no longer U6.6 (E3)
- net #A3: now also U6.2 (A1); no longer U1.8 (P3)
- net #CLK_CPU: now also U21.25 (CLK)
- net #D0: now also U21.19 (D0)
- net #D1: now also U21.20 (D1)
- net #D2: now also U21.1 (D2)
- net #D3: now also U21.40 (D3)
- net #D4: now also U21.39 (D4)
- net #D5: now also U21.38 (D5)
- net #D6: now also U21.3 (D6)
- net #D7: now also U21.2 (D7)
- net +12V: now also J8.b28 (+12V)
- net +5V: now also U6.6 (E3), J8.b1 (+5V), J8.b2 (+5V), J8.b3 (+5V), U21.26 (VCC)
- net -12V: now also J8.b29 (-12V)
- net /IOREQ: now also U1.8 (P3)
- net A0: now also J8.a7 (CA0)
- net A1: now also J8.a8 (CA1)
- net A10: now also J8.a17 (CA10)
- net A11: now also J8.a18 (CA11)
- net A12: now also J8.a19 (CA12)
- net A13: now also J8.a20 (CA13)
- net A14: now also J8.a21 (CA14)
- net A15: now also J8.a22 (CA15)
- net A16: now also J8.a25 (A16)
- net A17: now also J8.a26 (A17)
- net A18: now also J8.a27 (A18)
- net A19: now also J8.a28 (A19)
- net A2: now also J8.a9 (CA2)
- net A20: now also J8.a29 (A20)
- net A21: now also J8.a30 (A21)
- net A22/SCL: now also J8.a31 (SCL)
- net A23/SDA: now also J8.a32 (SDA)
- net A3: now also J8.a10 (CA3)
- net A4: now also J8.a11 (CA4)
- net A5: now also J8.a12 (CA5)
- net A6: now also J8.a13 (CA6)
- net A7: now also J8.a14 (CA7)
- net A8: now also J8.a15 (CA8)
- net A9: now also J8.a16 (CA9)
- net BUF_POTAX: now also U21.8 (PA6)
- net BUF_POTAY: now also U21.7 (PA7)
- net BUF_POTBX: now also U21.33 (PB6)
- net BUF_POTBY: now also U21.34 (PB7)
- net CLK_CPU: now also J8.b16 (CLK)
- net D0: now also J8.b7 (CD0)
- net D1: now also J8.b8 (CD1)
- net D2: now also J8.b9 (CD2)
- net D3: now also J8.b10 (CD3)
- net D4: now also J8.b11 (CD4)
- net D5: now also J8.b12 (CD5)
- net D6: now also J8.b13 (CD6)
- net D7: now also J8.b14 (CD7)
- net FIREA/LPA: now also U21.10 (PA4)
- net FIREB/LPB: now also U21.31 (PB4)
- net GND: now also J8.G (CHASSIS), J8.a1 (GND), J8.a2 (GND), J8.a3 (GND), J8.a4 (GND), J8.b32 (GND), U21.11 (GND)
- net JOYA0: now also U21.15 (PA0)
- net JOYA1: now also U21.14 (PA1)
- net JOYA2: now also U21.13 (PA2)
- net JOYA3: now also U21.12 (PA3)
- net JOYB0: now also U21.27 (PB0)
- net JOYB1: now also U21.28 (PB1)
- net JOYB2: now also U21.29 (PB2)
- net JOYB3: now also U21.30 (PB3)
- net MEMAQ: now also J8.a5 (MEMAQ)
- net ~{#IOREQ}: now also U21.36 (~{IORQ})
- net ~{#M1}: now also U21.37 (~{M1})
- net ~{#RD}: now also U21.35 (~{RD}); no longer U6.3 (A2)
- net ~{ADC_RDY}: now also U21.32 (PB5), U21.9 (PA5)
- net ~{BUSACK}: now also J8.a24 (~{BUSACK})
- net ~{BUSREQ}: now also J8.a23 (~{BUSREQ})
- net ~{HALT}: now also J8.b21 (~{HALT})
- net ~{INT0}: now also J8.b4 (~{INT0})
- net ~{INT1}: now also J8.b5 (~{INT1})
- net ~{INT2}: now also J8.b6 (~{INT2})
- net ~{INT3}: now also J8.a6 (~{INT3})
- net ~{INT}: now also J8.b17 (~{INT}), U21.23 (~{INT})
- net ~{IOREQ}: now also J8.b25 (~{IOREQ})
- net ~{M1}: now also J8.b19 (~{M1})
- net ~{MREQ}: now also J8.b24 (~{MREQ})
- net ~{NMI}: now also J8.b18 (~{NMI})
- net ~{RD_ADC}: now also U6.13 (O2); no longer U6.12 (O3)
- net ~{RD}: now also J8.b22 (~{RD})
- net ~{RESET}: now also J8.b15 (~{RESET})
- net ~{WAIT}: now also J8.b20 (~{WAIT})
- net ~{WR_MUX}: now also U6.12 (O3); no longer U6.9 (O6)
- net ~{WR}: now also J8.b23 (~{WR})
- net at U1.19 (P=R), U5.3, U6.4 (E1)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: now also U6.3 (A2)
- net at RN1.6 (R5), U1.9 (R3): no longer J2.2 (Pin_2)
- net IEI: now reaches IC1.6 (IEI)
- net IEI: now also J8.b26 (IEI)
- net IEO: now reaches IC1.7 (IEO)
- net IEO: now also J8.b27 (IEO)
- net ~{RD_PORTB} renamed ~{CS_PIO}
- no-connect marks 19 -> 28
Other:
- moved on the sheet: J2, J3, J4, J5, J6, LED1, R1, R3, R4, R5, RN1, U1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
