File: Modules/002-MIO Board V1/Schematics/Z80-MIO.kicad_sch (KiCad schematic)
At the start: 77 parts, among them J1 Conn_02x05_Odd_Even, J2 Conn_02x32_Row_Letter_First, J3 Conn_02x02_Top_Bottom, J4 Conn_02x06_Odd_Even, J5 Mini-DIN-6, J6 Mini-DIN-6, J7 Jumper_2_Bridged, J8 Conn_02x04_Odd_Even, J9 Conn_02x04_Odd_Even, Q1 BC548, U1 74HC688, U10 DS1307+, U11 74HC161, U12 Am9511A, U2 GAL16V8, U3 74HC2T45, U4 74HC245, U5 74HC245, U6 PIO-DIP-40, U7 7406, U8 PCF8584, U9 8048, Y1 32.768 kHz

Commit message: multiple updates
Parts:
- removed D10, D11, D12, D9: D, Diode_THT:D_DO-34_SOD68_P7.62mm_Horizontal, symbol Device:D
- removed D13: 5.1V, Diode_THT:D_DO-34_SOD68_P7.62mm_Horizontal, symbol Device:D_Zener
- removed J2: Conn_02x32_Row_Letter_First, Connector_DIN:DIN41612_Q_2x32_Male_Horizontal_THT, symbol Connector_Generic:Conn_02x32_Row_Letter_First
- added J10: Z8C_Card, Dennis:Z8C Card, symbol Dennis:Z8C_Card
- J4: value Conn_02x06_Odd_Even -> Conn_02x07_Odd_Even; footprint Connector_IDC:IDC-Header_2x06_P2.54mm_Latch_Horizontal -> Connector_IDC:IDC-Header_2x07_P2.54mm_Latch_Horizontal; symbol Connector_Generic:Conn_02x06_Odd_Even -> Connector_Generic:Conn_02x07_Odd_Even
- J5: footprint w_conn_av:PS2 -> Dennis:PS2
- J6: footprint w_conn_av:PS2 -> Dennis:PS2; symbol Connector:Mini-DIN-6 -> Dennis2:Mini-DIN-6_Shield
- R8, R9: value R -> 4k7
Connections:
- net +12V: now also J10.b28 (+12V)
- net +5V: now also U8.4 (~{IACK}), J10.b1 (+5V), J10.b2 (+5V), J10.b3 (+5V)
- net -12V: now also J10.b29 (-12V)
- net A0: now also J10.a7 (CA0)
- net A1: now also J10.a8 (CA1)
- net A10: now also J10.a17 (CA10)
- net A11: now also J10.a18 (CA11)
- net A12: now also J10.a19 (CA12)
- net A13: now also J10.a20 (CA13)
- net A14: now also J10.a21 (CA14)
- net A15: now also J10.a22 (CA15)
- net A16: now also J10.a25 (A16)
- net A17: now also J10.a26 (A17)
- net A18: now also J10.a27 (A18)
- net A19: now also J10.a28 (A19)
- net A2: now also J10.a9 (CA2)
- net A20: now also J10.a29 (A20)
- net A21: now also J10.a30 (A21)
- net A3: now also J10.a10 (CA3)
- net A4: now also J10.a11 (CA4)
- net A5: now also J10.a12 (CA5)
- net A6: now also J10.a13 (CA6)
- net A7: now also J10.a14 (CA7)
- net A8: now also J10.a15 (CA8)
- net A9: now also J10.a16 (CA9)
- net CLK_CPU: now also J10.b16 (CLK)
- net D0: now also J10.b7 (CD0)
- net D1: now also J10.b8 (CD1)
- net D2: now also J10.b9 (CD2)
- net D3: now also J10.b10 (CD3)
- net D4: now also J10.b11 (CD4)
- net D5: now also J10.b12 (CD5)
- net D6: now also J10.b13 (CD6)
- net D7: now also J10.b14 (CD7)
- net GND: now also J4.13 (Pin_13), J4.14 (Pin_14), J5.G, J6.G, J10.G (CHASSIS), J10.a1 (GND), J10.a2 (GND), J10.a3 (GND), J10.a4 (GND), J10.b32 (GND)
- net I2C_SCL: no longer J3.1 (Pin_1)
- net I2C_SDA: no longer J3.2 (Pin_2)
- net MEMAQ: now also J10.a5 (MEMAQ)
- net ~{#RESET}: no longer U8.19 (~{RST})
- net ~{#WR}: no longer U8.18 (~{WR})
- net ~{BUSACK}: now also J10.a24 (~{BUSACK})
- net ~{BUSREQ}: now also J10.a23 (~{BUSREQ})
- net ~{HALT}: now also J10.b21 (~{HALT})
- net ~{INT0}: now also J10.b4 (~{INT0})
- net ~{INT1}: now also J10.b5 (~{INT1})
- net ~{INT2}: now also J10.b6 (~{INT2})
- net ~{INT3}: now also J10.a6 (~{INT3})
- net ~{INT}: now also J10.b17 (~{INT})
- net ~{IOREQ}: now also J10.b25 (~{IOREQ})
- net ~{M1}: now also J10.b19 (~{M1})
- net ~{MREQ}: now also J10.b24 (~{MREQ})
- net ~{NMI}: now also J10.b18 (~{NMI})
- net ~{RD}: now also J10.b22 (~{RD})
- net ~{RESET}: now also J10.b15 (~{RESET})
- net ~{WAIT}: now also J10.b20 (~{WAIT})
- net ~{WR}: now also J10.b23 (~{WR})
- net FPU_CLK: now reaches J9.2 (Pin_2), J9.4 (Pin_4), J9.6 (Pin_6), J9.8 (Pin_8), U12.23 (CLK)
- net ~{INT_KB}: now reaches R1.2, U6.13 (PA2), U7.10, U7.12
- net SPK_DRV: now reaches R3.1, U6.12 (PA3)
- net ~{RST_IIC}: now reaches U6.14 (PA1)
- net ~{RST_IIC}: now also U8.19 (~{RST}); no longer U8.4 (~{IACK})
- net ~{INT_IIC}: now reaches R2.2, U6.15 (PA0), U8.5 (~{INT})
- net at U6.22 (IEO): now also J10.b27 (IEO)
- net at U6.24 (IEI): now also J10.b26 (IEI)
- net ~{CS_PIO}: now reaches U2.16 (IO4), U6.4 (~{CE})
- net ~{IIC_WR}: now reaches U2.14 (IO6)
- net ~{IIC_WR}: now also U8.18 (~{WR})
- net BOARD_CS: no longer names the net of U2.19 (IO1)
- net CS_FPU renamed ~{CS_FPU}
- net CS_IIC renamed ~{CS_IIC}
- net CS_PS2 renamed ~{CS_PS2}
- new net A22/SCL: J10.a31 (SCL), J3.1 (Pin_1)
- new net A23/SDA: J10.a32 (SDA), J3.2 (Pin_2)
- no-connect marks 24 -> 30
Other:
- note removed: "CS_PIO"
- moved on the sheet: BT1, C1, C10, C11, C12, C13, C14, C15, C16, C2, C3, C4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

Commit message: pushed updates
Parts:
- removed Q1: BC548, Package_TO_SOT_THT:TO-92_Inline, symbol Transistor_BJT:BC548
- removed R3: 220, Resistor_THT:R_Axial_DIN0204_L3.6mm_D1.6mm_P7.62mm_Horizontal, symbol Device:R
- removed U8: PCF8584, Package_DIP:DIP-20_W7.62mm_LongPads, symbol Interface_Expansion:PCF8584
- added IC1: CTC-DIP-28, Package_DIP:DIP-28_W15.24mm_LongPads, symbol Zilog_Z80_Peripherals:CTC-DIP-28
- added U13: 74LS74, symbol 74xx:74LS74
- added U7: 7406, Package_DIP:DIP-14_W7.62mm_Socket, symbol 74xx:74LS06
- added U8: 74S00, symbol 74xx:74LS00
- R2: value 10k -> 4k7
Connections:
- net A22 is gone; now on net A22/SCL: J3.3 (Pin_3)
- net A23 is gone; now on net A23/SDA: J3.4 (Pin_4)
- net ~{RST_IIC} is gone; now on net I2C_SCL: U6.14 (PA1)
- net #A0: now also IC1.18 (CS0)
- net #A1: now also IC1.19 (CS1)
- net #CLK_CPU: now also IC1.15 (CLK)
- net #D0: now also IC1.25 (D0), U13.12 (D)
- net #D1: now also IC1.26 (D1)
- net #D2: now also IC1.27 (D2)
- net #D3: now also IC1.28 (D3)
- net #D4: now also IC1.1 (D4)
- net #D5: now also IC1.2 (D5)
- net #D6: now also IC1.3 (D6)
- net #D7: now also IC1.4 (D7)
- net +5V: now also IC1.24 (+5V), U13.10 (~{S}), U13.14 (VCC), U13.4 (~{S}), U8.14 (VCC)
- net A22/SCL: no longer J3.1 (Pin_1)
- net A23/SDA: no longer J3.2 (Pin_2)
- net GND: now also IC1.5 (GND), U13.7 (GND), U8.7 (GND)
- net I2C_SCL: now also J3.1 (Pin_1)
- net I2C_SDA: now also J3.2 (Pin_2), U6.15 (PA0)
- net SPK_DRV: now also U13.9 (Q), U8.2; no longer U6.12 (PA3)
- net ~{#IOREQ}: now also IC1.10 (~{IORQ})
- net ~{#M1}: now also IC1.14 (~{M1})
- net ~{#RD}: now also IC1.6 (~{RD})
- net ~{#RESET}: now also IC1.17 (~{RESET}), U13.1 (~{R}), U8.4
- net ~{INT}: now also IC1.12 (~{INT})
- net PIO_PB0: now reaches J4.3 (Pin_3), R4.2
- net IEI_BUS: now reaches J10.b26 (IEI), U6.24 (IEI)
- net IEO_BUS: now reaches J10.b27 (IEO)
- net IEO_BUS: now also IC1.11 (IEO); no longer U6.22 (IEO)
- net PIO_PB7: now reaches J4.4 (Pin_4), R11.2
- net PIO_PB5: now reaches J4.8 (Pin_8), R13.2
- net PIO_PB6: now reaches J4.6 (Pin_6), R12.2
- net PIO_PB3: now reaches J4.9 (Pin_9), R7.2
- net PIO_PB2: now reaches J4.7 (Pin_7), R6.2
- net at LS1.2: now also U7.12
- net PIO_PB1: now reaches J4.5 (Pin_5), R5.2
- net CSQW: now reaches U10.7 (SQW/OUT)
- net CSQW: now also U6.12 (PA3), IC1.21 (CLK/TRG2), IC1.22 (CLK/TRG1), IC1.23 (CLK/TRG0)
- net PIO_PB4: now reaches J4.10 (Pin_10), R10.2
- net ~{CS_IIC} renamed ~{CS_CTC}
- net ~{CS_CTC}: now also IC1.16 (~{CE})
- net ~{IIC_WR} renamed ~{CS_BUZ}
- net ~{CS_BUZ}: now also U13.11 (C)
- net ~{INT_IIC} renamed ~{SPK_OFF}
- net ~{SPK_OFF}: now also U7.10, U8.5; no longer U6.15 (PA0)
- new net: U8.12, U8.13, U8.3
- new net: U8.10, U8.6, U8.9
- new net: U7.13, U8.11
- new net: U13.13 (~{R}), U8.8
- new net: IC1.20 (CLK/TRG3), IC1.9 (ZC/TO2)
- new net IEO_PIO: IC1.13 (IEI), U6.22 (IEO)
- new net SPK_FREQ: IC1.7 (ZC/TO0), U13.3 (C)
- new net SPK_FREQDIV2: U13.5 (Q), U8.1
- new net SPK_OFF: IC1.8 (ZC/TO1), U7.11
- new net ~{SPK_FREQDIV2}: U13.2 (D), U13.6 (~{Q})
Other:
- moved on the sheet: BT1, J3, LS1, R8, R9, U10, Y1
