File: Modules/004-Graphics Card V9958/Schematics/Z80-VDP.kicad_pcb (KiCad board)
At the start: 2 copper layers, 160 x 100.3 mm, 81 parts, among them J1 Conn_02x32_Row_Letter_First, J2 Conn_02x05_Counter_Clockwise, J4 S-VIDEO Out, J6 Composite Out, J7 RGBOut_Red, J8 RGBOut_Green, J9 RGBOut_Blue, U1 L7805, U10 41464, U11 CXA2075M, U12 41464, U13 41464, U14 41464, U15 41464, U2 74LS688, U3 74HC245, U4 74HC245, U5 74HC245, U6 74HC125, U7 74HC02, U8 V9958, U9 41464, X1 ACO-xxxMHz, Y1 21.477MHz

Commit message: multiple updates
Parts:
- removed the ? at (71.5, 147.6)
- removed H1: MountingHole_Pad, MountingHole:MountingHole_3.2mm_M3_DIN965_Pad
- added J3: Z8C_Card, Dennis:Z8C Card, F.Cu at (222.5, 102.9)
- J1: value Conn_02x32_Row_Letter_First -> Conn_02x04_Odd_Even; footprint Connector_DIN:DIN41612_Q_2x32_Male_Horizontal_THT -> Connector_PinHeader_2.54mm:PinHeader_2x04_P2.54mm_Vertical
- moved J1 39.7 mm to (181.6, 68.6), turned to 180 degrees
- moved C1 4.32 mm to (127.0, 91.7)
- moved U1 4.11 mm to (124.5, 83.2)
Connections:
- JP1 pad 2: unconnected-(JP1-Pad2) -> Net-(JP1-Pin_2)
- RN1 pad 7: Net-(RN1-Pad7) -> Net-(JP1-Pin_2)
- RN1 pad 8: unconnected-(RN1-Pad8) -> Net-(RN1-R7)
- U2 pad 4: /~{#M1} -> /~{#IOREQ}
- U2 pad 5: +5V -> Net-(RN1-R7)
- U2 pad 7: Net-(RN1-Pad7) -> Net-(JP1-Pin_2)
- U6 pad 10: (no net) -> GND
- U6 pad 11: (no net) -> unconnected-(U6-Pad11)
- U6 pad 12: (no net) -> GND
- U6 pad 13: (no net) -> GND
- U6 pad 4: (no net) -> GND
- U6 pad 5: (no net) -> GND
- U6 pad 6: (no net) -> unconnected-(U6-Pad6)
- U6 pad 8: (no net) -> unconnected-(U6-Pad8)
- U6 pad 9: (no net) -> GND
Routing:
- net +5V: track 508.7 -> 309.6 mm, vias 6 -> 4
- net GND: track 878.8 -> 710.4 mm, vias 7 -> 8
- net /~{#M1}: track 63.2 -> 0.00 mm, vias 2 -> 0
- net /~{INT3}: track 0.00 -> 57.9 mm, vias 0 -> 2
- net /~{INT2}: track 0.00 -> 49.6 mm, vias 0 -> 2
- net /~{INT1}: track 0.00 -> 46.1 mm, vias 0 -> 2
- net /~{INT0}: track 0.00 -> 39.7 mm
- net Net-(JP1-Pin_2): track 0.00 -> 36.1 mm, vias 0 -> 2
- net /AD0: track 84.0 -> 117.3 mm, vias 0 -> 1
- net /~{IRQ_OUT}: track 79.9 -> 106.4 mm, vias 1 -> 2
- net /#A7: track 31.6 -> 20.0 mm
- net Net-(RN1-R7): track 0.00 -> 11.1 mm, vias 0 -> 2
- net /~{#IOREQ}: track 59.7 -> 64.5 mm, vias 1 -> 5
- net Net-(U1-OUT): track 39.2 -> 43.5 mm
- net +12V: track 202.1 -> 198.0 mm
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Other:
- copper layers 2 -> 4
- board text added: "0"
- board text added: "1"
- board text added: "2"
- board text added: "3"
- board text added: "BANK X"
- board text added: "Color Video V1"
- board text added: "INT-CH"
- board text removed: "BANK 2"
- board text removed: "Color Video Controller V1"
