File: Modules/004-Graphics Card V9958/Schematics/Z80-VDP.kicad_sch (KiCad schematic)
At the start: 77 parts, among them J1 Conn_02x32_Row_Letter_First, J2 Conn_02x05_Counter_Clockwise, J4 S-VIDEO Out, J6 Composite Out, J7 RGBOut_Red, J8 RGBOut_Green, J9 RGBOut_Blue, U1 L7805, U10 41464, U11 CXA2075M, U12 41464, U13 41464, U14 41464, U15 41464, U2 74LS688, U3 74HC245, U4 74HC245, U5 74HC245, U6 74HC125, U7 74HC02, U8 V9958, U9 41464, X1 ACO-xxxMHz, Y1 21.477MHz

Commit message: multiple updates
Parts:
- removed J1: Conn_02x32_Row_Letter_First, Connector_DIN:DIN41612_Q_2x32_Male_Horizontal_THT, symbol Connector_Generic:Conn_02x32_Row_Letter_First
- added J3: Z8C_Card, Dennis:Z8C Card, symbol Dennis:Z8C_Card
- added J8: Conn_02x04_Odd_Even, Connector_PinHeader_2.54mm:PinHeader_2x04_P2.54mm_Vertical, symbol Connector_Generic:Conn_02x04_Odd_Even
- added unit 2 of U6
- added unit 3 of U6
- added unit 4 of U6
Connections:
- net /CAS1 is gone; now on net /CAS1: U8.60 (/CAS1)
- net +12V: now also J3.b28 (+12V)
- net +5V: now also J3.b1 (+5V), J3.b2 (+5V), J3.b3 (+5V); no longer U2.5 (R1)
- net -12V: now also J3.b29 (-12V)
- net /CAS0: no longer U8.61 (/CAS0)
- net /RAS: no longer U8.62 (/RAS)
- net A0: now also J3.a7 (CA0)
- net A1: now also J3.a8 (CA1)
- net A10: now also J3.a17 (CA10)
- net A11: now also J3.a18 (CA11)
- net A12: now also J3.a19 (CA12)
- net A13: now also J3.a20 (CA13)
- net A14: now also J3.a21 (CA14)
- net A15: now also J3.a22 (CA15)
- net A16: now also J3.a25 (A16)
- net A17: now also J3.a26 (A17)
- net A18: now also J3.a27 (A18)
- net A19: now also J3.a28 (A19)
- net A2: now also J3.a9 (CA2)
- net A20: now also J3.a29 (A20)
- net A21: now also J3.a30 (A21)
- net A22/SCL: now also J3.a31 (SCL)
- net A23/SDA: now also J3.a32 (SDA)
- net A3: now also J3.a10 (CA3)
- net A4: now also J3.a11 (CA4)
- net A5: now also J3.a12 (CA5)
- net A6: now also J3.a13 (CA6)
- net A7: now also J3.a14 (CA7)
- net A8: now also J3.a15 (CA8)
- net A9: now also J3.a16 (CA9)
- net CLK_CPU: now also J3.b16 (CLK)
- net D0: now also J3.b7 (CD0)
- net D1: now also J3.b8 (CD1)
- net D2: now also J3.b9 (CD2)
- net D3: now also J3.b10 (CD3)
- net D4: now also J3.b11 (CD4)
- net D5: now also J3.b12 (CD5)
- net D6: now also J3.b13 (CD6)
- net D7: now also J3.b14 (CD7)
- net GND: now also J3.G (CHASSIS), J3.a1 (GND), J3.a2 (GND), J3.a3 (GND), J3.a4 (GND), J3.b32 (GND), U6.10, U6.12, U6.13, U6.4, U6.5, U6.9
- net MEMAQ: now also J3.a5 (MEMAQ)
- net R/W: no longer U8.57 (R/W)
- net ~{#IOREQ}: now also U2.4 (P1)
- net ~{#M1}: no longer U2.4 (P1)
- net ~{BUSACK}: now also J3.a24 (~{BUSACK})
- net ~{BUSREQ}: now also J3.a23 (~{BUSREQ})
- net ~{HALT}: now also J3.b21 (~{HALT})
- net ~{INT0}: now also J3.b4 (~{INT0}), J8.1 (Pin_1)
- net ~{INT1}: now also J3.b5 (~{INT1}), J8.3 (Pin_3)
- net ~{INT2}: now also J3.b6 (~{INT2}), J8.5 (Pin_5)
- net ~{INT3}: now also J3.a6 (~{INT3}), J8.7 (Pin_7)
- net ~{INT}: now also J3.b17 (~{INT})
- net ~{IOREQ}: now also J3.b25 (~{IOREQ})
- net ~{IRQ_OUT}: now also J8.2 (Pin_2), J8.4 (Pin_4), J8.6 (Pin_6), J8.8 (Pin_8)
- net ~{M1}: now also J3.b19 (~{M1})
- net ~{MREQ}: now also J3.b24 (~{MREQ})
- net ~{NMI}: now also J3.b18 (~{NMI})
- net ~{RD}: now also J3.b22 (~{RD})
- net ~{RESET}: now also J3.b15 (~{RESET})
- net ~{WAIT}: now also J3.b20 (~{WAIT})
- net ~{WR}: now also J3.b23 (~{WR})
- net at RN1.7 (R6), U2.7 (R2): now also JP1.2 (Pin_2)
- net at RN1.8 (R7): now also U2.5 (R1)
- new net: J3.b26 (IEI), J3.b27 (IEO)
- new net R/W: U8.57 (R/W)
- new net /CAS0: U8.61 (/CAS0)
- new net /RAS: U8.62 (/RAS)
- no-connect marks 6 -> 8
Other:
- note added: "Bank 0"
- note added: "Bank 1"
- note added: "Bank X"
- moved on the sheet: C1, C2, C27, C28, C29, C30, C31, C32, C33, C34, C5, C6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

Commit message: pushed updates
Connections:
- net +5VA: now also C13.1, C14.1; no longer C13.2, C14.2
- net GNDA: now also C13.2, C14.2; no longer C13.1, C14.1
Other:
- moved on the sheet: C13, C14
Changed lines of the file:
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@@
     )
   )
-  (symbol (lib_id "Device:C_Polarized") (at 232.41 187.96 180) (unit 1)
-    (in_bom yes) (on_board yes) (dnp no)
-    (property "Reference" "C14" (at 229.87 185.42 0)
+  (symbol (lib_id "Device:C_Polarized") (at 232.41 187.96 0) (mirror y) (unit 1)
+    (in_bom yes) (on_board yes) (dnp no)
+    (property "Reference" "C14" (at 229.87 190.5 0)
       (effects (font (size 1.27 1.27)) (justify right))
     )
-    (property "Value" "47uF" (at 236.22 190.5 90)
+    (property "Value" "47uF" (at 236.22 185.42 90)
       (effects (font (size 1.27 1.27)) (justify right))
     )
-    (property "Footprint" "Capacitor_THT:CP_Radial_D6.3mm_P2.50mm" (at 231.4448 184.15 0)
+    (property "Footprint" "Capacitor_THT:CP_Radial_D6.3mm_P2.50mm" (at 231.4448 191.77 0)
       (effects (font (size 1.27 1.27)) hide)
     )
@@
     )
   )
-  (symbol (lib_id "Device:C_Polarized") (at 232.41 127 180) (unit 1)
-    (in_bom yes) (on_board yes) (dnp no)
-    (property "Reference" "C13" (at 229.87 124.46 0)
+  (symbol (lib_id "Device:C_Polarized") (at 232.41 127 0) (mirror y) (unit 1)
+    (in_bom yes) (on_board yes) (dnp no)
+    (property "Reference" "C13" (at 229.87 129.54 0)
       (effects (font (size 1.27 1.27)) (justify right))
     )
-    (property "Value" "47uF" (at 236.22 129.54 90)
+    (property "Value" "47uF" (at 236.22 124.46 90)
       (effects (font (size 1.27 1.27)) (justify right))
     )
-    (property "Footprint" "Capacitor_THT:CP_Radial_D6.3mm_P2.50mm" (at 231.4448 123.19 0)
-      (effects (font (size 1.27 1.27)) hide)
-    )
+    (property "Footprint" "Capacitor_THT:CP_Radial_D6.3mm_P2.50mm" (at 231.4448 130.81 0)
+      (effects (font (size 1.27 1.27)) hide)
+    )

Commit message: several fixes
Parts:
- U6: value 74HC125 -> 74LS125
Connections:
- net /CAS0: now also U10.16 (~{CAS}), U9.16 (~{CAS}); no longer U10.5 (~{RAS}), U9.5 (~{RAS})
- net /RAS: now also U10.5 (~{RAS}), U12.5 (~{RAS}), U13.5 (~{RAS}), U14.5 (~{RAS}), U15.5 (~{RAS}), U9.5 (~{RAS}); no longer U10.16 (~{CAS}), U12.16 (~{CAS}), U13.16 (~{CAS}), U14.16 (~{CAS}), U15.16 (~{CAS}), U9.16 (~{CAS})
- net /CAS1: now also U12.16 (~{CAS}), U13.16 (~{CAS}); no longer U12.5 (~{RAS}), U13.5 (~{RAS})
- net /CASX: now also U14.16 (~{CAS}), U15.16 (~{CAS}); no longer U14.5 (~{RAS}), U15.5 (~{RAS})
Other:
- note added: "74LS125 or 74HCT125 V9958 TTL Levels not compatible with HC"
Changed lines of the file:
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@@
     (effects (font (size 1.27 1.27)) (justify left bottom))
   )
+  (text "74LS125 or 74HCT125\nV9958 TTL Levels not compatible with HC"
+    (at 317.5 240.03 0)
+    (effects (font (size 1.27 1.27)) (justify left bottom))
+  )
   (text "Bank X" (at 327.66 102.87 0)
     (effects (font (size 1.27 1.27)) (justify left bottom))
@@
     (effects (font (size 1.524 1.524)) (justify left bottom))
   )
-  (label "/CAS0" (at 226.06 95.25 0) (fields_autoplaced)
+  (label "/CAS0" (at 226.06 97.79 0) (fields_autoplaced)
     (effects (font (size 1.524 1.524)) (justify left bottom))
   )
@@
     (effects (font (size 1.524 1.524)) (justify left bottom))
   )
-  (label "/CAS0" (at 226.06 53.34 0) (fields_autoplaced)
+  (label "/CAS0" (at 226.06 55.88 0) (fields_autoplaced)
     (effects (font (size 1.524 1.524)) (justify left bottom))
   )
@@
     (effects (font (size 1.524 1.524)) (justify left bottom))
   )
-  (label "{slash}CASX" (at 314.96 53.34 0) (fields_autoplaced)
+  (label "{slash}CASX" (at 314.96 55.88 0) (fields_autoplaced)
     (effects (font (size 1.524 1.524)) (justify left bottom))
   )
@@
     (effects (font (size 1.27 1.27)) (justify left bottom))
   )
-  (label "{slash}CAS1" (at 270.51 53.34 0) (fields_autoplaced)
+  (label "{slash}CAS1" (at 270.51 55.88 0) (fields_autoplaced)
     (effects (font (size 1.524 1.524)) (justify left bottom))
   )
@@
     (effects (font (size 1.524 1.524)) (justify left bottom))
   )
-  (label "{slash}CAS1" (at 270.51 95.25 0) (fields_autoplaced)
+  (label "{slash}CAS1" (at 270.51 97.79 0) (fields_autoplaced)
     (effects (font (size 1.524 1.524)) (justify left bottom))
   )
@@
     (effects (font (size 1.27 1.27)) (justify left bottom))
   )
-  (label "/RAS" (at 270.51 55.88 0) (fields_autoplaced)
+  (label "/RAS" (at 270.51 53.34 0) (fields_autoplaced)
     (effects (font (size 1.524 1.524)) (justify left bottom))
   )
@@
     (effects (font (size 1.27 1.27)) (justify left bottom))
   )
-  (label "{slash}CASX" (at 314.96 95.25 0) (fields_autoplaced)
+  (label "{slash}CASX" (at 314.96 97.79 0) (fields_autoplaced)
     (effects (font (size 1.524 1.524)) (justify left bottom))
   )
@@
     (effects (font (size 1.27 1.27)) (justify right bottom))
   )
-  (label "/RAS" (at 226.06 97.79 0) (fields_autoplaced)
+  (label "/RAS" (at 226.06 95.25 0) (fields_autoplaced)
     (effects (font (size 1.524 1.524)) (justify left bottom))
   )
@@
     (effects (font (size 1.27 1.27)) (justify right bottom))
   )
-  (label "/RAS" (at 314.96 55.88 0) (fields_autoplaced)
+  (label "/RAS" (at 314.96 53.34 0) (fields_autoplaced)
     (effects (font (size 1.524 1.524)) (justify left bottom))
   )
@@
     (effects (font (size 1.27 1.27)) (justify right bottom))
   )
-  (label "/RAS" (at 314.96 97.79 0) (fields_autoplaced)
+  (label "/RAS" (at 314.96 95.25 0) (fields_autoplaced)
     (effects (font (size 1.524 1.524)) (justify left bottom))
   )
@@
     (effects (font (size 1.524 1.524)) (justify left bottom))
   )
-  (label "/RAS" (at 270.51 97.79 0) (fields_autoplaced)
+  (label "/RAS" (at 270.51 95.25 0) (fields_autoplaced)
     (effects (font (size 1.524 1.524)) (justify left bottom))
   )
@@
     (effects (font (size 1.524 1.524)) (justify left bottom))
   )
-  (label "/RAS" (at 226.06 55.88 0) (fields_autoplaced)
+  (label "/RAS" (at 226.06 53.34 0) (fields_autoplaced)
     (effects (font (size 1.524 1.524)) (justify left bottom))
   )
@@
       (effects (font (size 1.27 1.27)))
     )
-    (property "Value" "74HC125" (at 316.23 217.17 0)
+    (property "Value" "74LS125" (at 316.23 217.17 0)
       (effects (font (size 1.27 1.27)))
     )
@@
       (effects (font (size 1.27 1.27)) (justify left))
     )
-    (property "Value" "74HC125" (at 187.325 255.2699 0)
+    (property "Value" "74LS125" (at 187.325 255.2699 0)
       (effects (font (size 1.27 1.27)) (justify left))
     )
@@
       (effects (font (size 1.27 1.27)))
     )
-    (property "Value" "74HC125" (at 387.35 207.01 0)
+    (property "Value" "74LS125" (at 387.35 207.01 0)
       (effects (font (size 1.27 1.27)))
     )
@@
       (effects (font (size 1.27 1.27)))
     )
-    (property "Value" "74HC125" (at 387.35 224.79 0)
+    (property "Value" "74LS125" (at 387.35 224.79 0)
       (effects (font (size 1.27 1.27)))
     )
@@
       (effects (font (size 1.27 1.27)))
     )
-    (property "Value" "74HC125" (at 387.35 242.57 0)
+    (property "Value" "74LS125" (at 387.35 242.57 0)
       (effects (font (size 1.27 1.27)))
     )
