File: Modules/005-Z80-Sound/z80-SOUND.kicad_sch (KiCad schematic)
At the start: 25 parts, among them IC1 SIO0-DIP-40, J2 Conn_02x05_Odd_Even, J6 DIN-5, J7 DIN-5, J8 Z8C_Card, U1 74LS688, U10 74HC590, U14 74HCT04, U18 6N137, U2 74HC245, U3 74HC245, U4 74HC245, U5 74HC02, U6 74HC138, U7 SN76489AN, U8 YM2612, X1 1MHz

Commit message: pushed updates
Parts:
- removed J2: Conn_02x05_Odd_Even, Connector_PinHeader_2.54mm:PinHeader_2x05_P2.54mm_Vertical, symbol Connector_Generic:Conn_02x05_Odd_Even
- removed J6, J7: DIN-5, w_conn_av:din-5, symbol Connector:DIN-5
- removed JP1: Jumper_3_Open, Connector_PinHeader_2.54mm:PinHeader_1x03_P2.54mm_Vertical, symbol Jumper:Jumper_3_Open
- removed LED1: MENOTR_A500_Dual_3mm, w_conn_av:MENTOR A500 Dual 3mm, symbol CustomSymbols:MENOTR_A500_Dual_3mm
- removed RN1: R_Network08, Resistor_THT:R_Array_SIP9, symbol Device:R_Network08
- removed unit 5 of U14
- removed unit 2 of U14
- removed U18: 6N137, Package_DIP:DIP-8_W7.62mm, symbol Isolator:6N137
- added C1, C14, C15, C16, C2, C20, C21, C22, C23, C24, C25, C26, C27, C3, C4, C5, C7: 100nF, Capacitor_THT:C_Rect_L7.0mm_W2.0mm_P5.00mm, symbol Device:C_Small
- added C10, C11: 10uF, Capacitor_THT:CP_Radial_D6.3mm_P2.50mm, symbol Device:C_Polarized
- added C12, C13, C6: 2n2, Capacitor_THT:C_Rect_L7.0mm_W2.0mm_P5.00mm, symbol Device:C_Small
- added C17, C18, C19: 220uF, Capacitor_THT:CP_Radial_D8.0mm_P3.50mm, symbol Device:C_Polarized
- added C8, C9: 1u, Capacitor_THT:CP_Radial_D6.3mm_P2.50mm, symbol Device:C_Polarized
- added D1, D2, D3, D4: 1N4148, Diode_THT:D_DO-35_SOD27_P7.62mm_Horizontal, symbol Diode:1N4148
- added D5, D6, D7, D8: 5.1V, Diode_THT:D_DO-34_SOD68_P7.62mm_Horizontal, symbol Device:D_Zener
- added FB1, FB2: FerriteBead, Resistor_THT:R_Axial_DIN0414_L11.9mm_D4.5mm_P15.24mm_Horizontal, symbol Device:FerriteBead
- added J2, J7: Conn_01x16, Connector_PinSocket_2.54mm:PinSocket_1x16_P2.54mm_Vertical, symbol Connector_Generic:Conn_01x16
- added J3: OutL, Dennis:RCA_Reichelt, symbol Connector:Conn_Coaxial
- added J4: OutR, Dennis:RCA_Reichelt, symbol Connector:Conn_Coaxial
- added J5: DB15, Connector_Dsub:DSUB-15_Female_Horizontal_P2.77x2.84mm_EdgePinOffset9.90mm_Housed_MountingHolesOffset11.32mm, symbol Connector:DA15_Plug_MountingHoles
- added J6: Conn_02x04_Odd_Even, Connector_PinHeader_2.54mm:PinHeader_2x04_P2.54mm_Vertical, symbol Connector_Generic:Conn_02x04_Odd_Even
- added Q1, Q2, Q3: 2N3904, Package_TO_SOT_THT:TO-92_Inline, symbol Transistor_BJT:2N3904
- added R10, R11, R13, R14: 2k2, Resistor_THT:R_Axial_DIN0204_L3.6mm_D1.6mm_P7.62mm_Horizontal, symbol Device:R
- added R12, R15, R16, R17, R18, R25, R26, R27, R6, R7, R8, R9: 1k, Resistor_THT:R_Axial_DIN0204_L3.6mm_D1.6mm_P7.62mm_Horizontal, symbol Device:R
- added R19, R20, R21, R22: 100R, Resistor_THT:R_Axial_DIN0204_L3.6mm_D1.6mm_P7.62mm_Horizontal, symbol Device:R
- added R23, R24: 10k, Resistor_THT:R_Axial_DIN0204_L3.6mm_D1.6mm_P7.62mm_Horizontal, symbol Device:R
- added RN1, RN3: R_Network04, Resistor_THT:R_Array_SIP5, symbol Device:R_Network04
- added RN2: 3-103J, Resistor_THT:R_Array_SIP8, symbol Device:R_Pack04_SIP_Split
- added RN4: R_Network04, Resistor_THT:R_Array_SIP9, symbol Device:R_Network08
- added RV1, RV2, RV3, RV4, RV5: 10K, Potentiometer_THT:Potentiometer_Bourns_3299W_Vertical, symbol Device:R_Potentiometer_Trim
- added SW1: MONO_SW, Dennis:DPDT_Vertical, symbol Switch:SW_SPDT
- added U11: TL074, Package_DIP:DIP-14_W7.62mm_Socket, symbol Amplifier_Operational:TL074
- added U12: 74LS125, Package_DIP:DIP-14_W7.62mm_Socket, symbol 74xx:74LS125
- added unit 7 of U13
- added unit 6 of U13
- added unit 5 of U13
- added U14: 74LS00, Package_DIP:DIP-14_W7.62mm_Socket, symbol 74xx:74LS00
- added U15, U16: 6N137, Package_DIP:DIP-8_W7.62mm, symbol Isolator:6N137
- added U17: L78L09_TO92, Package_TO_SOT_THT:TO-92_Inline, symbol Regulator_Linear:L78L09_TO92
- added U18: L79L09_TO92, Package_TO_SOT_THT:TO-92_Inline, symbol Regulator_Linear:L79L05_TO92
- added U19: ~, Connector_PinSocket_2.54mm:PinSocket_1x07_P2.54mm_Vertical, symbol Dennis2:SI5351_Module
- added unit 2 of U7
- added unit 5 of U7
- added unit 3 of U7
- added U9: AY-3-8910, Package_DIP:DIP-40_W15.24mm_Socket, symbol oldchips:AY-3-8912
- R1, R2, R3, R4, R5: value 10k -> 1k
- U13: renamed from U14; value 74HCT04 -> 74LS04; footprint (none) -> Package_DIP:DIP-14_W7.62mm_Socket
- U5: renamed from U8; footprint (none) -> Package_DIP:DIP-24_W15.24mm_Socket
- U6: renamed from U7; footprint Package_DIP:DIP-16_W7.62mm -> Package_DIP:DIP-16_W7.62mm_Socket
- U7: renamed from U5; value 74HC02 -> 74LS02; footprint Package_DIP:DIP-14_W7.62mm_Socket_LongPads -> Package_DIP:DIP-14_W7.62mm_Socket
- renumbered J8 to J1, U6 to U8
Connections:
- net /IOREQ is gone; now on net ~{#IOREQ}: U1.2 (P0), U1.4 (P1), U1.6 (P2), U1.8 (P3)
- net ~{CS_PIO} is gone; now on net ~{CS_YM}: U8.14 (O1)
- net ~{RD_ADC} is gone; now on net ~{CS_SN}: U8.13 (O2)
- net #A0: now also U5.17 (A0), J7.9 (Pin_9), U7.5
- net #A1: now also U5.18 (A1), J7.10 (Pin_10)
- net #A2: now also J7.11 (Pin_11)
- net #A3: now also J7.12 (Pin_12)
- net #A4: now also J7.13 (Pin_13)
- net #A5: now also J7.14 (Pin_14)
- net #A6: now also J7.15 (Pin_15)
- net #A7: now also J7.16 (Pin_16)
- net #CLK_CPU: now also J2.8 (Pin_8)
- net #D0: now also J7.1 (Pin_1), U9.37 (DA0)
- net #D1: now also J7.2 (Pin_2), U9.36 (DA1)
- net #D2: now also J7.3 (Pin_3), U9.35 (DA2)
- net #D3: now also J7.4 (Pin_4), U9.34 (DA3)
- net #D4: now also J7.5 (Pin_5), U9.33 (DA4)
- net #D5: now also J7.6 (Pin_6), U9.32 (DA5)
- net #D6: now also J7.7 (Pin_7), U9.31 (DA6)
- net #D7: now also J7.8 (Pin_8), U9.30 (DA7)
- net +12V: now also U17.3 (VI)
- net +5V: now also C1.1, C2.1, C20.1, C21.1, C22.1, C23.1, C24.1, C25.1, C26.1, C27.1, C3.1, C4.1, C5.1, C7.1, FB2.1, J2.11 (Pin_11), J6.1 (Pin_1), J6.3 (Pin_3), J6.5 (Pin_5), J6.7 (Pin_7), R23.1, R24.1, RN2.4 (R2.2), RN2.8 (R4.2), RN3.1 (common), RN4.1 (common), U12.14 (VCC), U13.14 (VCC), U14.14 (VCC), U15.7 (EN), U15.8 (VCC), U16.7 (EN), U16.8 (VCC), U19.1 (VIN), U7.14 (VCC), U9.25 (A8), U9.28 (BC2), U9.40 (VCC); no longer R1.1, R3.2, R4.2, R5.1
- net -12V: now also U18.2 (VI)
- net A22/SCL: now also J2.9 (Pin_9), U19.3 (SDA)
- net A23/SDA: now also J2.10 (Pin_10), U19.4 (SCL)
- net GND: now also U1.3 (R0), U1.5 (R1), U1.7 (R2), U1.9 (R3), C1.2, C2.2, C20.2, C21.2, C22.2, C23.2, C24.2, C25.2, C26.2, C27.2, C3.2, C4.2, C5.2, C7.2, D1.2 (A), D2.2 (A), D3.2 (A), D4.2 (A), D5.2 (A), D6.2 (A), D7.2 (A), D8.2 (A), FB1.1, J2.3 (Pin_3), J5.0 (PAD), J5.1, J5.11 (P111), J5.5, Q1.1 (E), Q2.1 (E), Q3.1 (E), R13.2, R14.2, RN1.1 (common), U12.7 (GND), U13.7 (GND), U14.12, U14.13, U14.7 (GND), U15.5 (GND), U16.5 (GND), U19.2 (GND), U7.7 (GND), U9.1 (GND), U9.24 (/A9)
- net ~{#IOREQ}: now also J2.4 (Pin_4)
- net ~{#RD}: now also J2.6 (Pin_6)
- net ~{#RESET}: now also J2.5 (Pin_5), U9.23 (/RESET)
- net ~{#WR}: now also J2.7 (Pin_7), U7.8
- net at R3.1: now also R4.1, RV3.2
- net AUDIO_MIX_L: now reaches R1.2
- net AUDIO_MIX_L: now also R4.2, J2.1 (Pin_1), R6.2, R7.1, SW1.3 (C), U11.2 (-)
- net at U13.6: now also RN2.2 (R1.2)
- net ~{CS_YM}: now reaches U5.14 (CS)
- net GNDA: now reaches U5.19 (AGND)
- net GNDA: now also C14.2, C15.2, C16.1, C17.2, C18.2, C19.1, FB1.2, J2.13 (Pin_13), J2.16 (Pin_16), J3.2 (Ext), J4.2 (Ext), RV1.3, RV2.3, RV3.3, RV4.1, RV5.1, U11.3 (+), U11.5 (+), U17.2 (GND), U18.1 (GND)
- net OUT_YM_R: now reaches U5.20 (MOR)
- net OUT_YM_R: now also C9.1
- net OUT_YM_L: now reaches U5.21 (MOL)
- net OUT_YM_L: now also C8.1
- net +5VA: now reaches U5.22 (AVcc)
- net +5VA: now also C14.1, C17.1, FB2.2, J2.12 (Pin_12)
- net #~{CLK_YM}: now reaches U5.24 (CLOCK_IN)
- net #~{CLK_YM}: now also Q2.3 (C), RN3.3 (R2)
- net at U13.8: now also U13.5
- net at U1.18 (R7): now also J6.8 (Pin_8), RN1.2 (R1)
- net at U1.16 (R6): now also J6.6 (Pin_6), RN1.3 (R2)
- net at U1.14 (R5): now also J6.4 (Pin_4), RN1.4 (R3)
- net at U1.12 (R4): now also J6.2 (Pin_2), RN1.5 (R4)
- net AUDIO_MIX_R: now reaches R5.2
- net AUDIO_MIX_R: now also R2.2, R3.2, J2.2 (Pin_2), R8.1, SW1.2 (B), U11.6 (-)
- net MIDI_OUT/~{THRU}: now reaches U13.1
- net MIDI_OUT/~{THRU}: now also IC1.24 (~{RTSB}), U14.10
- net at U13.2: now also U14.5; no longer R2.1
- net MIDIB_TX: now reaches IC1.26 (TXDB)
- net MIDIB_TX: now also U13.9
- net MIDIB_RX: now reaches IC1.28 (RXDB)
- net MIDIB_RX: now also U13.12
- net #~{CLK_SN}: now reaches U6.14 (CLOCK)
- net #~{CLK_SN}: now also Q1.3 (C), RN3.2 (R1)
- net ~{CS_SN}: now reaches U6.6 (~{CE})
- net at U6.7 (AUDIO_OUT): now also C6.1
- net MIDI_IN renamed MIDIA_RX
- net MIDIA_RX: now also U13.10, U14.9; no longer U13.5
- net MIDI_OUT renamed MIDIA_TX
- net MIDIA_TX: now also U14.4; no longer U13.9
- net ~{WR_MUX} renamed ~{CS_PSG}
- net ~{CS_PSG}: now also U7.6, U7.9
- new net: R16.1, R20.1, U12.6
- new net: U14.1, U14.6
- new net: Q1.2 (B), R25.2
- new net: RN4.2 (R1), U12.13, U9.6 (IOB7)
- new net: RN4.3 (R2), U12.10, U9.7 (IOB6)
- new net: RN4.4 (R3), U12.4, U9.8 (IOB5)
- new net: RN4.5 (R4), U12.1, U9.9 (IOB4)
- new net: RN4.6 (R5), U12.12, U9.10 (IOB3)
- new net: RN4.7 (R6), U12.9, U9.11 (IOB2)
- new net: RN4.8 (R7), U12.5, U9.12 (IOB1)
- new net: RN4.9 (R8), U12.2, U9.13 (IOB0)
- new net: Q2.2 (B), R26.2
- new net: D3.1 (K), D7.1 (K), R17.2, U9.19 (IOA2)
- new net: D2.1 (K), D6.1 (K), R16.2, U9.20 (IOA1)
- new net: R18.1, R22.1, U12.11
- new net: R17.1, R21.1, U12.8
- new net: R10.1, R11.1, U9.3 (A_CHB)
- new net: C13.2, R11.2, R12.2, R14.1
- new net: R5.1, RV5.2
- new net: R24.2, U13.13, U16.6 (VO)
- new net: Q3.2 (B), R27.2
- new net: C9.2, RV2.1
- new net: R2.1, RV2.2
- new net: C8.2, RV1.1
- new net: R1.1, RV1.2
- new net: C6.2, RV3.1
- new net: C10.1, R7.2, U11.1
- new net: C10.2, J3.1 (In)
- new net: D1.1 (K), D5.1 (K), R15.2, U9.21 (IOA0)
- new net: C13.1, U11.12 (+)
- new net: D4.1 (K), D8.1 (K), R18.2, U9.18 (IOA3)
- new net: U7.10, U9.27 (BDIR)
- new net: U7.4, U9.29 (BC1)
- new net: R12.1, U9.38 (A_CHC)
- new net: R9.1, U9.4 (A_CHA)
- new net: C12.2, R10.2, R13.1, R9.2
- new net: C12.1, U11.10 (+)
- new net: R15.1, R19.1, U12.3
- new net: C11.1, R8.2, U11.7
- new net: R6.1, RV4.2
- new net: RV5.3, U11.13 (-), U11.14
- new net: R23.2, U13.11, U15.6 (VO)
- new net: U14.2, U14.8
- new net: RV4.3, U11.8, U11.9 (-)
- new net: C11.2, J4.1 (In)
- new net: RN2.6 (R3.2), U14.3
- new net #~{CLK_PSG}: Q3.3 (C), RN3.4 (R3), U9.22 (CLOCK)
- new net +9VA: C15.1, C18.1, J2.15 (Pin_15), U11.4 (V+), U17.1 (VO)
- new net -9VA: C16.2, C19.2, J2.14 (Pin_14), U11.11 (V-), U18.3 (VO)
- new net CLK_PSG: R27.1, U19.5 (CLK2)
- new net CLK_SN: R25.1, U19.7 (CLK0)
- new net CLK_YM: R26.1, U19.6 (CLK1)
- new net MIDIA_IN_DATA: J5.8, U15.3 (C)
- new net MIDIA_IN_VCC: J5.15 (P15), U15.2 (A)
- new net MIDIA_OUT_DATA: J5.6, RN2.5 (R3.1)
- new net MIDIA_OUT_VCC: J5.13 (P13), RN2.7 (R4.1)
- new net MIDIB_IN_DATA: J5.7, U16.3 (C)
- new net MIDIB_IN_VCC: J5.14 (P14), U16.2 (A)
- new net MIDIB_OUT_DATA: J5.12 (P12), RN2.1 (R1.1)
- new net MIDIB_OUT_VCC: J5.4, RN2.3 (R2.1)
- new net TRIG_OUT_A: J5.3, R19.2
- new net TRIG_OUT_B: J5.10 (P10), R20.2
- new net TRIG_OUT_C: J5.2, R21.2
- new net TRIG_OUT_D: J5.9 (P9), R22.2
- no-connect marks 23 -> 38
Other:
- note removed: "MIDI-IN"
- note removed: "MIDI-OUT"
- title: Z8C Midi Interfacee -> Z8C Audio Interface
- moved on the sheet: U13A, U13C, U13D, U5, U6

Commit message: several fixes
Connections:
- no-connect marks 38 -> 39
