File: Modules/005-Z80-Sound/z80-SOUND_rev1.kicad_sch (KiCad schematic)
At the start: 105 parts, among them IC1 SIO0-DIP-40, J1 Z8C_Card, J2 Conn_01x16, J3 OutL, J4 OutR, J5 DB15, J6 Conn_02x04_Odd_Even, J7 Conn_01x16, Q1 2N3904, Q2 2N3904, Q3 2N3904, SW1 MONO_SW, U1 74HC688, U10 74HC590, U11 TL074, U12 74LS125, U13 74LS04, U14 74LS00, U15 6N137, U16 6N137, U17 L78L09_TO92, U18 L79L09_TO92, U2 74HTC245, U3 74HC245, U4 74HC245, U5 YM2612, U6 SN76489AN, U7 74HC02, U8 74HC138, U9 AY-3-8910, X1 1MHz

Commit message: fix Sound board rev1
Parts:
- removed Q1, Q2, Q3: 2N3904, Package_TO_SOT_THT:TO-92_Inline, symbol Transistor_BJT:2N3904
- removed R25, R26, R27: 1k, Resistor_THT:R_Axial_DIN0204_L3.6mm_D1.6mm_P7.62mm_Horizontal, symbol Device:R
- removed RN3: R_Network04, Resistor_THT:R_Array_SIP5, symbol Device:R_Network04
- C12, C13: value 2n2 -> 10n
- C15, C16: value 100nF -> 1uF
- C18, C19: value 220uF -> 100uF
- C6: footprint Capacitor_THT:C_Rect_L7.0mm_W2.0mm_P5.00mm -> Capacitor_THT:C_Rect_L7.0mm_W3.5mm_P5.00mm
- D5, D6, D7, D8: footprint Diode_THT:D_DO-34_SOD68_P7.62mm_Horizontal -> Diode_THT:D_DO-35_SOD27_P7.62mm_Horizontal
- RN2: value 3-103J -> 3-102J
Connections:
- net CLK_PSG is gone; now on net #~{CLK_PSG}: U19.5 (CLK2)
- net CLK_SN is gone; now on net #~{CLK_SN}: U19.7 (CLK0)
- net CLK_YM is gone; now on net #~{CLK_YM}: U19.6 (CLK1)
- net A22/SCL: now also U19.4 (SCL); no longer U19.3 (SDA)
- net A23/SDA: now also U19.3 (SDA); no longer U19.4 (SCL)
- no-connect marks 39 -> 38
Other:
- note removed: "Level shifter not working and not required after all. Wired SI5351 outputs directly to corresponding Ppins on RN3. Removed Q1,Q2,Q3,RN3,R25,R25,R27"
- note removed: "Pin 3/4 swapped!!!"
