File: Modules/007-MemoryExpansion/007-MemoryExpansion.kicad_pcb (KiCad board)
At the start: 2 copper layers, 160 x 100.3 mm, 1 part, among them J1 Z8C_Card

Commit message: several fixes
Parts:
- added J2: ENA19, Connector_PinHeader_2.54mm:PinHeader_2x01_P2.54mm_Vertical, F.Cu at (156.2, 73.7)
- added JP1: Conn_02x06_Odd_Even, Connector_PinHeader_2.54mm:PinHeader_2x06_P2.54mm_Vertical, F.Cu at (116.1, 147.7)
- added R1: 4.7k, Resistor_THT:R_Axial_DIN0204_L3.6mm_D1.6mm_P2.54mm_Vertical, F.Cu at (158.8, 78.7)
- added RN1: 4k7, Resistor_THT:R_Array_SIP5, F.Cu at (186.7, 99.1)
- added RN2: R_Network08, Resistor_THT:R_Array_SIP9, F.Cu at (157.2, 151.9)
- added SW1: SW_DIP_x04, Package_DIP:DIP-8_W7.62mm_Socket, F.Cu at (175.3, 100.3)
- added U1: 74LS157, Package_DIP:DIP-16_W7.62mm, F.Cu at (87.6, 80.0)
- added U10: 74LS245, Package_DIP:DIP-20_W7.62mm, F.Cu at (151.1, 21.6)
- added U11: ~, Package_DIP:DIP-24_W15.24mm, F.Cu at (138.4, 80.0)
- added U12: ~, Package_DIP:DIP-20_W7.62mm_Socket, F.Cu at (87.6, 21.6)
- added U13: ~, Package_DIP:DIP-20_W7.62mm_Socket, F.Cu at (100.3, 21.6)
- added U15: 74LS74, Package_DIP:DIP-14_W7.62mm, F.Cu at (151.1, 50.8)
- added U16: ~, Package_DIP:DIP-20_W7.62mm_Socket, F.Cu at (87.6, 50.8)
- added U17: ~, Package_DIP:DIP-20_W7.62mm_Socket, F.Cu at (100.3, 50.8)
- added U18: 74LS125, Package_DIP:DIP-14_W7.62mm, F.Cu at (175.3, 80.0)
- added U19: ~, Package_DIP:DIP-20_W7.62mm_Socket, F.Cu at (113.0, 21.6)
- added U2: 74LS157, Package_DIP:DIP-16_W7.62mm, F.Cu at (101.0, 80.0)
- added U20: ~, Package_DIP:DIP-20_W7.62mm_Socket, F.Cu at (125.7, 21.6)
- added U21: 74LS138, Package_DIP:DIP-16_W7.62mm, F.Cu at (88.9, 113.0)
- added U22: ~, Package_DIP:DIP-20_W7.62mm_Socket, F.Cu at (113.0, 50.8)
- added U23: ~, Package_DIP:DIP-20_W7.62mm_Socket, F.Cu at (125.7, 50.8)
- added U24: 74LS175, Package_DIP:DIP-16_W7.62mm, F.Cu at (125.7, 80.0)
- added U3: 74LS157, Package_DIP:DIP-16_W7.62mm, F.Cu at (113.7, 80.0)
- added U4: ~, Package_DIP:DIP-24_W7.62mm_Socket, F.Cu at (163.2, 80.0)
- added U5: 74LS688, Package_DIP:DIP-20_W7.62mm, F.Cu at (187.7, 120.3)
- added U6: 74LS245, Package_DIP:DIP-20_W7.62mm, F.Cu at (138.4, 21.6)
- added U7: 74LS374, Package_DIP:DIP-20_W7.62mm, F.Cu at (138.4, 50.8)
- added U8: 74LS157, Package_DIP:DIP-16_W7.62mm, F.Cu at (115.6, 113.0)
- added U9: ~, Package_DIP:DIP-24_W7.62mm_Socket, F.Cu at (163.2, 45.7)
- added X1: 40MHz, Oscillator:Oscillator_DIP-14, F.Cu at (182.9, 72.4)
- J1: value Z8C_Card -> Z8C_Ca#RD
- moved J1 32.9 mm to (230.5, 67.5)
