File: Modules/007-MemoryExpansion/007-MemoryExpansion.kicad_sch (KiCad schematic)
At the start: 30 parts, among them J1 Z8C_Card, J2 CTC_CLK_SEL, J3 ENA19, U1 74LS157, U10 74LS157, U11 74LS245, U15 74LS01, U19 74LS595, U2 74LS157, U20 74LS04, U24 74LS138, U27 74LS02, U3 74LS157, U4 74LS74, U5 74LS02, U6 74LS688, U7 74LS125, U8 74LS139, U9 74LS374, X1 25MHz

Commit message: several fixes
Parts:
- removed J2: CTC_CLK_SEL, Connector_PinHeader_2.54mm:PinHeader_2x04_P2.54mm_Vertical, symbol Connector_Generic:Conn_02x04_Odd_Even
- removed J3: ENA19, Connector_PinHeader_2.54mm:PinHeader_2x01_P2.54mm_Vertical, symbol Connector_Generic:Conn_01x02
- removed U1, U2, U3: 74LS157, Package_DIP:DIP-16_W7.62mm, symbol 74xx:74LS157
- removed U13, U14, U16, U17, U21, U22, U25, U26: ~, Package_DIP:DIP-20_W7.62mm_Socket, symbol Dennis2:HY534256A
- removed U15: 74LS01, symbol 74xx:74LS01
- removed U19: 74LS595, Package_DIP:DIP-16_W7.62mm, symbol 74xx:74LS595
- removed U20: 74LS04, Package_DIP:DIP-14_W7.62mm, symbol 74xx:74LS04
- removed U24: 74LS138, Package_DIP:DIP-16_W7.62mm, symbol 74xx:74LS138
- removed U27, U5: 74LS02, Package_DIP:DIP-14_W7.62mm, symbol 74xx:74LS02
- removed unit 2 of U4
- removed unit 1 of U4
- removed U8: 74LS139, Package_DIP:DIP-16_W7.62mm, symbol 74xx:74LS139
- removed X1: 25MHz, Oscillator:Oscillator_DIP-14, symbol Oscillator:ACO-xxxMHz
- added JP1: Conn_02x06_Odd_Even, Connector_PinHeader_2.54mm:PinHeader_2x06_P2.54mm_Vertical, symbol Connector_Generic:Conn_02x06_Odd_Even
- added R2: 10k, symbol Device:R
- added RN1: 4k7, Resistor_THT:R_Array_SIP5, symbol Device:R_Network04
- added RN2: R_Network08, Resistor_THT:R_Array_SIP9, symbol Device:R_Network08
- added SW1: SW_DIP_x04, Package_DIP:DIP-8_W7.62mm_Socket, symbol Switch:SW_DIP_x04
- added U1, U2, U3: 74F257, symbol 74xx:74LS257
- added U12, U6: 74LS245, Package_DIP:DIP-20_W7.62mm, symbol 74xx:74LS245
- added U13, U9: ~, Dennis:SIMM, symbol Dennis2:SIMM30P
- added U14: 74LS01, symbol 74xx:74LS01
- added U21, U4: ~, Package_DIP:DIP-24_W7.62mm_Socket, symbol Dennis2:GAL22V10
- added U24: 74LS175, Package_DIP:DIP-16_W7.62mm, symbol 74xx:74LS175
- added U25: 74LS139, symbol 74xx:74LS139
- added U26: 74F195, symbol 74xx:74LS195
- added U27: ~, Package_DIP:DIP-24_W15.24mm, symbol Dennis2:TMM2016B
- added X2: 50MHz, Oscillator:Oscillator_DIP-14, symbol Oscillator:ACO-xxxMHz
- J1: value Z8C_Card -> Z8C_Ca#RD
- R1: value 4.7k -> 10k; footprint Resistor_THT:R_Axial_DIN0204_L3.6mm_D1.6mm_P2.54mm_Vertical -> (none)
- renumbered U11 to U10, U12 to U11, U4 to U15, U7 to U18, U6 to U5, U9 to U7, U10 to U8
Connections:
- net +5V: now also JP1.1 (Pin_1), JP1.11 (Pin_11), JP1.3 (Pin_3), JP1.5 (Pin_5), JP1.7 (Pin_7), JP1.9 (Pin_9), SW1.1, SW1.2, SW1.3, SW1.4, U12.20 (VCC), U13.1 (Vcc), U13.30 (Vcc), U21.24 (VCC), U24.1 (~{Mr}), U24.16 (VCC), U26.16 (VCC), U26.9 (~{PE}), U27.24 (Vcc), U4.24 (VCC), U6.20 (VCC), U9.1 (Vcc), U9.30 (Vcc), X2.14 (Vcc)
- net GND: now also R1.1, U5.1 (G), R2.1, RN1.1 (common), RN2.1 (common), U1.15 (OE), U12.10 (GND), U13.22 (GND), U13.9 (GND), U2.15 (OE), U21.12 (GND), U24.8 (GND), U26.4 (P0), U26.5 (P1), U26.6 (P2), U26.7 (P3), U26.8 (GND), U27.12 (GND), U27.18 (~{CS}), U27.19 (A10), U27.20 (~{OE}), U3.15 (OE), U4.12 (GND), U6.10 (GND), U9.22 (GND), U9.9 (GND), X2.7 (GND); no longer R1.2, U11.22 (A9), U11.23 (A8)
- net JENA19: no longer R1.1
- net MBA12: now also U1.3 (I1a)
- net MBA13: now also U1.6 (I1b)
- net MBA14: now also U1.13 (I1c)
- net MBA15: now also U1.10 (I1d)
- net MBA16: now also U2.3 (I1a)
- net MBA17: now also U2.6 (I1b)
- net MBA18: now also U2.13 (I1c), U21.9 (I9)
- net MBA19: now also U10.11 (B7), U11.17 (D7), U2.10 (I1d), U21.11 (I11)
- net MBPROT: now also U12.12 (B6), U27.16 (D6), U4.16 (IO16); no longer U10.11 (B7), U11.17 (D7)
- net MDA0: now also U13.3 (DQ0), U6.18 (B0), U9.3 (DQ0)
- net MDA1: now also U13.6 (DQ1), U6.17 (B1), U9.6 (DQ1)
- net MDA2: now also U13.10 (DQ2), U6.16 (B2), U9.10 (DQ2)
- net MDA3: now also U13.13 (DQ3), U6.15 (B3), U9.13 (DQ3)
- net MDA4: now also U13.16 (DQ4), U6.14 (B4), U9.16 (DQ4)
- net MDA5: now also U13.20 (DQ5), U6.13 (B5), U9.20 (DQ5)
- net MDA6: now also U13.23 (DQ6), U6.12 (B6), U9.23 (DQ6)
- net MDA7: now also U13.25 (QP), U6.11 (B7), U9.25 (QP)
- net MMA0: now also U1.4 (Za), U13.4 (A0), U9.4 (A0)
- net MMA1: now also U1.7 (Zb), U13.5 (A1), U9.5 (A1)
- net MMA2: now also U1.12 (Zc), U13.7 (A2), U9.7 (A2)
- net MMA3: now also U1.9 (Zd), U13.8 (A3), U9.8 (A3)
- net MMA4: now also U13.11 (A4), U2.4 (Za), U9.11 (A4)
- net MMA5: now also U13.12 (A5), U2.7 (Zb), U9.12 (A5)
- net MMA6: now also U13.14 (A6), U2.12 (Zc), U9.14 (A6)
- net MMA7: now also U13.15 (A7), U2.9 (Zd), U9.15 (A7)
- net MMA8: now also U13.17 (A8), U3.4 (Za), U9.17 (A8)
- net MPROTEN: now also U7.19 (O7), U4.15 (IO15)
- net REGBNK0: now also U7.2 (O0), U27.4 (A4); no longer U7.12 (O4)
- net REGBNK1: now also U7.5 (O1), U27.3 (A5); no longer U7.15 (O5)
- net REGBNK2: now also U7.6 (O2), U27.2 (A6); no longer U7.16 (O6)
- net REGBNK3: now also U7.9 (O3), U27.1 (A7); no longer U7.19 (O7)
- net REGMAP0: now also U24.2 (Q0); no longer U7.2 (O0)
- net REGMAP1: now also U24.7 (Q1); no longer U7.5 (O1)
- net REGMAP2: now also U24.10 (Q2); no longer U7.6 (O2)
- net REGMAP3: now also U24.15 (Q3); no longer U7.9 (O3)
- net ~{CSMAP}: now also U4.20 (IO20); no longer U10.19 (CE)
- net ~{REFRSH}: now also U21.11 (I11)
- net ~{WRMAP}: now also U4.21 (IO21); no longer U11.21 (R/~{W})
- net ~{NMIGAT}: now reaches U18.4
- net ~{NMIGAT}: now also U4.14 (IO14)
- net at U11.5 (A3), U8.12 (Zd): now also U27.5 (A3)
- net at U11.6 (A2), U8.9 (Zc): now also U27.6 (A2)
- net at U11.7 (A1), U8.7 (Zb): now also U27.7 (A1)
- net at U11.8 (A0), U8.4 (Za): now also U27.8 (A0)
- net ~{RDPROT}: now reaches U18.1
- net ~{RDPROT}: now also U4.18 (IO18)
- net at U5.12 (R4): now also JP1.6 (Pin_6), RN2.5 (R4)
- net at U5.14 (R5): now also JP1.8 (Pin_8), RN2.4 (R3)
- net at U5.16 (R6): now also JP1.10 (Pin_10), RN2.3 (R2)
- net at U5.18 (R7): now also JP1.12 (Pin_12), RN2.2 (R1)
- net at U5.3 (R0): now also RN2.9 (R8)
- net at U5.5 (R1): now also RN2.8 (R7)
- net at U5.7 (R2): now also JP1.2 (Pin_2), RN2.7 (R6)
- net at U5.9 (R3): now also JP1.4 (Pin_4), RN2.6 (R5)
- net CA12 renamed #CA12
- net CA13 renamed #CA13
- net CA14 renamed #CA14
- net #CA14: now also U4.11 (I11)
- net CA15 renamed #CA15
- net #CA15: now also U4.13 (I13/~{OE})
- net CA2 renamed #CA2
- net #CA2: now also U1.14 (I0c)
- net CA3 renamed #CA3
- net #CA3: now also U1.11 (I0d)
- net CA4 renamed #CA4
- net #CA4: now also U2.2 (I0a)
- net CA5 renamed #CA5
- net #CA5: now also U2.5 (I0b)
- net CA6 renamed #CA6
- net #CA6: now also U2.14 (I0c)
- net CA7 renamed #CA7
- net #CA7: now also U2.11 (I0d)
- net CD0 renamed #CD0
- net #CD0: now also U12.2 (A0), U24.4 (D0), U6.2 (A0)
- net CD1 renamed #CD1
- net #CD1: now also U12.3 (A1), U24.5 (D1), U6.3 (A1)
- net CD2 renamed #CD2
- net #CD2: now also U12.4 (A2), U24.12 (D2), U6.4 (A2)
- net CD3 renamed #CD3
- net #CD3: now also U12.5 (A3), U24.13 (D3), U6.5 (A3)
- net CD4 renamed #CD4
- net #CD4: now also U12.6 (A4), U6.6 (A4)
- net CD5 renamed #CD5
- net #CD5: now also U12.7 (A5), U6.7 (A5)
- net CD6 renamed #CD6
- net #CD6: now also U12.8 (A6), U6.8 (A6)
- net CD7 renamed #CD7
- net #CD7: now also U12.9 (A7), U6.9 (A7)
- net ~{IOREQ} renamed ~{#IOREQ}
- net ~{#IOREQ}: now also U4.5 (I5)
- net ~{WRREG} renamed WRPROT
- net WRPROT: now also U4.19 (IO19)
- net ~{WR} renamed ~{#WR}
- net ~{#WR}: now also U12.1 (A->B), U13.21 (~{WE}), U4.8 (I8), U6.1 (A->B), U9.21 (~{WE})
- new net: R2.2, U12.11 (B7)
- new net: U26.10 (CP), X2.8 (OUT)
- new net: RN1.5 (R4), SW1.5, U4.1 (I1/CLK)
- new net: RN1.4 (R3), SW1.6, U4.2 (I2)
- new net: RN1.3 (R2), SW1.7, U4.3 (I3)
- new net: RN1.2 (R1), SW1.8, U4.4 (I4)
- new net: R1.2, U27.17 (D7)
- new net #CA0: U1.2 (I0a), U4.9 (I9)
- new net #CA1: U1.5 (I0b), U4.11 (I11)
- new net #CA10: U3.14 (I0c)
- new net #CA11: U3.11 (I0d)
- new net #CA8: U3.2 (I0a)
- new net #CA9: U3.5 (I0b)
- new net DRAMTIM: U21.22 (IO22), U26.2 (J), U26.3 (~{K})
- new net MBA20: U12.18 (B0), U27.9 (D0), U3.3 (I1a)
- new net MBA21: U12.17 (B1), U27.10 (D1), U3.6 (I1b)
- new net MBA22: U12.16 (B2), U21.4 (I4), U27.11 (D2), U3.13 (I1c)
- new net MBA23: U12.15 (B3), U21.5 (I5), U27.13 (D3), U3.10 (I1d)
- new net MBA24: U12.14 (B4), U21.6 (I6), U27.14 (D4)
- new net MBA25: U12.13 (B5), U21.7 (I7), U27.15 (D5)
- new net MDP: U13.29 (DP), U9.29 (DP)
- new net MFULL: U4.17 (IO17), U7.16 (O6)
- new net MMA10: U13.19 (A10), U3.12 (Zc), U9.19 (A10)
- new net MMA11: U13.24 (A11), U3.9 (Zd), U9.24 (A11)
- new net MMA9: U13.18 (A9), U3.7 (Zb), U9.18 (A9)
- new net MQP: U13.25 (QP), U9.25 (QP)
- new net REGBNK4: U11.23 (A8), U27.23 (A8), U7.12 (O4)
- new net REGBNK5: U11.22 (A9), U27.22 (A9), U7.15 (O5)
- new net SQCAS: U21.3 (I3), U26.13 (Q2)
- new net SQCLR: U21.23 (IO23), U26.1 (~{MR})
- new net SQMUX: U1.1 (S), U2.1 (S), U21.2 (I2), U26.14 (Q1), U3.1 (S)
- new net SQRAS: U21.1 (I1/CLK), U26.15 (Q0)
- new net WRREG: U24.9 (Cp), U4.22 (IO22)
- new net ~{#MREQ}: U4.6 (I6)
- new net ~{#RD}: U4.7 (I7)
- new net ~{#RESET}: U21.8 (I8)
- new net ~{CSMAP0}: U10.19 (CE)
- new net ~{CSMAP1}: U12.19 (CE)
- new net ~{CS_ROM0}: U21.18 (IO18)
- new net ~{CS_ROM1}: U21.19 (IO19)
- new net ~{CS_SRAM}: U21.20 (IO20)
- new net ~{DRAMREQ}: U21.13 (I13/~{OE}), U4.23 (IO23), U6.19 (CE)
- new net ~{MCAS0}: U21.15 (IO15), U9. (~{CASP}), U9.2 (~{CAS})
- new net ~{MCAS1}: U13. (~{CASP}), U13.2 (~{CAS}), U21.17 (IO17)
- new net ~{MRAS0}: U21.14 (IO14), U9.27 (~{RAS})
- new net ~{MRAS1}: U13.27 (~{RAS}), U21.16 (IO16)
- new net ~{WRMAP0}: U11.21 (R/~{W})
- new net ~{WRMAP1}: U27.21 (R/~{W})
- no-connect marks 3 -> 2
Other:
- note added: "Base address select"
- note added: "Current Page Protected"
- note added: "DRAM Memory range selected"
- note added: "Enable Memory Protection"
- note added: "Map Memory Multiplexer"
- note added: "Read Protect Enabled"
- note added: "Trigger NMI"
- note added: "Write Bank Register"
- note added: "Write Config Register"
- note added: "Write Map RAM"
- note removed: "90ns"
- note removed: "MREQ Triggered"
- note removed: "Mapper propagation delay ~100ns"
- note removed: "RAS before CAS Refresh generator"
- note removed: "TRIGGER NMI ON ILLEGAL ACCESS"
- moved on the sheet: U10, U11, U18A, U18B, U5, U7, U8
