File: Modules/007-MemoryExpansion/_autosave-007-MemoryExpansion.kicad_pcb (KiCad board)
At the start: 2 copper layers, 160 x 100.3 mm, 30 parts, among them J1 Z8C_Card, J2 CTC_CLK_SEL, J3 ENA19, U1 74LS157, U10 74LS157, U11 74LS245, U19 74LS595, U2 74LS157, U20 74LS04, U23 74LS06, U24 74LS138, U27 74LS02, U3 74LS157, U4 74LS74, U5 74LS02, U6 74LS688, U7 74LS125, U8 74LS139, U9 74LS374, X1 25MHz

Commit message: several fixes
Parts:
- removed J3: ENA19, Connector_PinHeader_2.54mm:PinHeader_2x01_P2.54mm_Vertical
- removed U14, U25, U26: ~, Package_DIP:DIP-20_W7.62mm_Socket
- added JP1: Conn_02x06_Odd_Even, Connector_PinHeader_2.54mm:PinHeader_2x06_P2.54mm_Vertical, F.Cu at (116.1, 147.7)
- added RN1: 4k7, Resistor_THT:R_Array_SIP5, F.Cu at (186.7, 99.1)
- added RN2: R_Network08, Resistor_THT:R_Array_SIP9, F.Cu at (157.2, 151.9)
- added SW1: SW_DIP_x04, Package_DIP:DIP-8_W7.62mm_Socket, F.Cu at (175.3, 100.3)
- added U15: 74LS74, Package_DIP:DIP-14_W7.62mm, F.Cu at (151.1, 50.8)
- added U18: 74LS125, Package_DIP:DIP-14_W7.62mm, F.Cu at (175.3, 80.0)
- added X2: 50MHz, Oscillator:Oscillator_DIP-14, F.Cu at (314.2, 73.7)
- J1: value Z8C_Card -> Z8C_Ca#RD
- J2: value CTC_CLK_SEL -> ENA19; footprint Connector_PinHeader_2.54mm:PinHeader_2x04_P2.54mm_Vertical -> Connector_PinHeader_2.54mm:PinHeader_2x01_P2.54mm_Vertical
- U10: value 74LS157 -> 74LS245; footprint Package_DIP:DIP-16_W7.62mm -> Package_DIP:DIP-20_W7.62mm
- U11: value 74LS245 -> ~; footprint Package_DIP:DIP-20_W7.62mm -> Package_DIP:DIP-24_W15.24mm
- U12: value ~ -> 74LS245; footprint Package_DIP:DIP-24_W15.24mm -> Package_DIP:DIP-20_W7.62mm
- U13: footprint Package_DIP:DIP-20_W7.62mm_Socket -> Dennis:SIMM
- U19: value 74LS595 -> ~; footprint Package_DIP:DIP-16_W7.62mm -> Package_DIP:DIP-20_W7.62mm_Socket
- U20: value 74LS04 -> ~; footprint Package_DIP:DIP-14_W7.62mm -> Package_DIP:DIP-20_W7.62mm_Socket
- U21: footprint Package_DIP:DIP-20_W7.62mm_Socket -> Package_DIP:DIP-24_W7.62mm_Socket
- U23: value 74LS06 -> ~; footprint Package_DIP:DIP-14_W7.62mm -> Package_DIP:DIP-20_W7.62mm_Socket
- U24: value 74LS138 -> 74LS175
- U27: value 74LS02 -> ~; footprint Package_DIP:DIP-14_W7.62mm -> Package_DIP:DIP-24_W15.24mm
- U4: value 74LS74 -> ~; footprint Package_DIP:DIP-14_W7.62mm -> Package_DIP:DIP-24_W7.62mm_Socket
- U5: value 74LS02 -> 74LS688; footprint Package_DIP:DIP-14_W7.62mm -> Package_DIP:DIP-20_W7.62mm
- U6: value 74LS688 -> 74LS245
- U7: value 74LS125 -> 74LS374; footprint Package_DIP:DIP-14_W7.62mm -> Package_DIP:DIP-20_W7.62mm
- U8: value 74LS139 -> 74LS157
- U9: value 74LS374 -> ~; footprint Package_DIP:DIP-20_W7.62mm -> Dennis:SIMM
- X1: value 25MHz -> 40MHz
- moved U27 120.9 mm to (293.9, 64.8)
- moved U9 103.9 mm to (158.2, -15.0)
- moved U13 92.4 mm to (158.2, -5.33)
- moved U21 87.8 mm to (88.9, 113.0), turned to 90 degrees
- moved U23 85.5 mm to (125.7, 50.8)
- moved U10 74.0 mm to (151.1, 21.6)
- moved R1 70.1 mm to (158.8, 78.7), turned to -90 degrees
- moved U12 68.7 mm to (87.6, 21.6)
- moved U5 66.7 mm to (187.7, 120.3)
- moved U8 57.8 mm to (115.6, 113.0), turned to 90 degrees
- moved X1 54.8 mm to (182.9, 72.4), turned to 90 degrees
- moved U19 37.0 mm to (113.0, 21.6)
- moved J2 33.1 mm to (156.2, 73.7), turned to 0 degrees
- moved U20 32.4 mm to (125.7, 21.6)
- moved U22 26.5 mm to (113.0, 50.8)
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Connections:
- net /CA10 renamed /#CA10
- net /CA11 renamed /#CA11
- J2 pad 1: unconnected-(J2-Pin_1-Pad1) -> +5V
- J2 pad 2: unconnected-(J2-Pin_2-Pad2) -> /JENA19
- U1 pad 11: /CA2 -> /#CA2
- U1 pad 14: /CA3 -> /#CA3
- U1 pad 2: /CA0 -> /#CA0
- U1 pad 5: /CA1 -> /#CA1
- U10 pad 1: /~{CSMAP} -> /~{#WR}
- U10 pad 10: /CA14 -> GND
- U10 pad 11: /REGMAP2 -> /MBA19
- U10 pad 12: Net-(U10-Zd) -> /MBA18
- U10 pad 13: /CA15 -> /MBA17
- U10 pad 14: /REGMAP3 -> /MBA16
- U10 pad 15: GND -> /MBA15
- U10 pad 16: +5V -> /MBA14
- U10 pad 2: /REGMAP0 -> /#CD0
- U10 pad 3: /CA12 -> /#CD1
- U10 pad 4: Net-(U10-Za) -> /#CD2
- U10 pad 5: /REGMAP1 -> /#CD3
- U10 pad 6: /CA13 -> /#CD4
- U10 pad 7: Net-(U10-Zb) -> /#CD5
- U10 pad 8: GND -> /#CD6
- U10 pad 9: Net-(U10-Zc) -> /#CD7
- U11 pad 1: /~{WR} -> /REGBNK3
- U11 pad 10: GND -> /MBA13
- U11 pad 11: /MBPROT -> /MBA14
- U11 pad 12: /MBA18 -> GND
- U11 pad 13: /MBA17 -> /MBA15
- U11 pad 15: /MBA15 -> /MBA17
- U11 pad 16: /MBA14 -> /MBA18
- U11 pad 17: /MBA13 -> /MBA19
- U11 pad 18: /MBA12 -> GND
- U11 pad 19: /~{CSMAP} -> GND
- U11 pad 2: /CD0 -> /REGBNK2
- U11 pad 20: +5V -> GND
- U11 pad 3: /CD1 -> /REGBNK1
- U11 pad 4: /CD2 -> /REGBNK0
- U11 pad 5: /CD3 -> Net-(U11-A3)
- U11 pad 6: /CD4 -> Net-(U11-A2)
- U11 pad 7: /CD5 -> Net-(U11-A1)
- U11 pad 8: /CD6 -> Net-(U11-A0)
- U11 pad 9: /CD7 -> /MBA12
- U12 pad 1: /REGBNK3 -> /~{#WR}
- U12 pad 10: /MBA13 -> GND
- U12 pad 11: /MBA14 -> Net-(U12-B7)
- U12 pad 12: GND -> /MBPROT
- U12 pad 13: /MBA15 -> /MBA25
- U12 pad 14: /MBA16 -> /MBA24
- U12 pad 15: /MBA17 -> /MBA23
- U12 pad 16: /MBA18 -> /MBA22
- U12 pad 17: /MBPROT -> /MBA21
- U12 pad 18: GND -> /MBA20
- U12 pad 19: GND -> /~{CSMAP1}
- U12 pad 2: /REGBNK2 -> /#CD0
- U12 pad 20: GND -> +5V
- U12 pad 3: /REGBNK1 -> /#CD1
- U12 pad 4: /REGBNK0 -> /#CD2
- U12 pad 5: Net-(U10-Zd) -> /#CD3
- U12 pad 6: Net-(U10-Zc) -> /#CD4
- U12 pad 7: Net-(U10-Zb) -> /#CD5
- U12 pad 8: Net-(U10-Za) -> /#CD6
- U12 pad 9: /MBA12 -> /#CD7
- U13 pad 1: /MDA0 -> +5V
- U13 pad 10: GND -> /MDA2
- U13 pad 13: /MMA6 -> /MDA3
- U13 pad 14: /MMA7 -> /MMA6
- U13 pad 15: /MMA8 -> /MMA7
- U13 pad 16: /~{DBANK1_RD} -> /MDA4
- U13 pad 17: /~{MCAS} -> /MMA8
- U13 pad 18: /MDA2 -> /MMA9
- U13 pad 19: /MDA3 -> /MMA10
- U13 pad 2: /MDA1 -> /~{MCAS1}
- U13 pad 20: +5V -> /MDA5
- U13 pad 3: /~{DBANK1_WR} -> /MDA0
- U13 pad 4: /~{MRAS} -> /MMA0
- U13 pad 5: (no net) -> /MMA1
- U13 pad 6: /MMA0 -> /MDA1
- U13 pad 7: /MMA1 -> /MMA2
- U13 pad 8: /MMA2 -> /MMA3
- U13 pad 9: /MMA3 -> GND
- U19 pad 1: /~{MCASR} -> /MDA0
- U19 pad 10: +5V -> GND
- U19 pad 11: Net-(U19-RCLK) -> /MMA4
- U19 pad 12: Net-(U19-RCLK) -> /MMA5
- U19 pad 13: /~{MREQ} -> /MMA6
- U19 pad 14: /~{MREQ} -> /MMA7
- U19 pad 15: /~{MMUX} -> /MMA8
- U19 pad 16: +5V -> /~{DBANK3_RD}
- U19 pad 2: unconnected-(U19-QC-Pad2) -> /MDA1
- U19 pad 3: unconnected-(U19-QD-Pad3) -> /~{DBANK3_WR}
- U19 pad 4: unconnected-(U19-QE-Pad4) -> /~{MRAS}
- U19 pad 5: unconnected-(U19-QF-Pad5) -> (no net)
- U19 pad 6: unconnected-(U19-QG-Pad6) -> /MMA0
- U19 pad 7: unconnected-(U19-QH-Pad7) -> /MMA1
- U19 pad 8: GND -> /MMA2
- U19 pad 9: unconnected-(U19-QH'-Pad9) -> /MMA3
- U2 pad 11: /CA6 -> /#CA6
- U2 pad 14: /CA7 -> /#CA7
- U2 pad 2: /CA4 -> /#CA4
- U2 pad 5: /CA5 -> /#CA5
- U20 pad 1: /~{REFRSH} -> /MDA0
- U20 pad 10: unconnected-(U20-Pad10) -> GND
- U20 pad 11: unconnected-(U20-Pad11) -> /MMA4
- U20 pad 12: unconnected-(U20-Pad12) -> /MMA5
- U20 pad 13: unconnected-(U20-Pad13) -> /MMA6
- U20 pad 14: unconnected-(U20G-VCC-Pad14) -> /MMA7
- U20 pad 2: /MUXEN -> /MDA1
- U20 pad 3: /MUXEN -> /~{DBANK4_WR}
- U20 pad 4: Net-(U15-Pad3) -> /~{MRAS}
- U20 pad 5: unconnected-(U20-Pad5) -> (no net)
- U20 pad 6: unconnected-(U20-Pad6) -> /MMA0
- U20 pad 7: unconnected-(U20G-GND-Pad7) -> /MMA1
- U20 pad 8: unconnected-(U20-Pad8) -> /MMA2
- U20 pad 9: unconnected-(U20-Pad9) -> /MMA3
- U21 pad 1: /MDA0 -> /SQRAS
- U21 pad 10: GND -> (no net)
- U21 pad 11: /MMA4 -> /MBA19
- U21 pad 12: /MMA5 -> GND
- U21 pad 13: /MMA6 -> /~{DRAMREQ}
- U21 pad 14: /MMA7 -> /~{MRAS0}
- U21 pad 15: /MMA8 -> /~{MCAS0}
- U21 pad 16: /~{DBANK3_RD} -> /~{MRAS1}
- U21 pad 17: /~{MCAS} -> /~{MCAS1}
- U21 pad 18: /MDA2 -> /~{CS_ROM0}
- U21 pad 19: /MDA3 -> /~{CS_ROM1}
- U21 pad 2: /MDA1 -> /SQMUX
- U21 pad 20: +5V -> /~{CS_SRAM}
- U21 pad 3: /~{DBANK3_WR} -> /SQCAS
- U21 pad 4: /~{MRAS} -> /MBA22
- U21 pad 5: (no net) -> /MBA23
- U21 pad 6: /MMA0 -> /MBA24
- U21 pad 7: /MMA1 -> /MBA25
- U21 pad 8: /MMA2 -> /~{#RESET}
- U21 pad 9: /MMA3 -> /MBA18
- U22 pad 1: /MDA0 -> /MDA4
- U22 pad 16: /~{DBANK4_RD} -> /~{DBANK3_RD}
- U22 pad 18: /MDA2 -> /MDA6
- U22 pad 19: /MDA3 -> /MDA7
- U22 pad 2: /MDA1 -> /MDA5
- U22 pad 3: /~{DBANK4_WR} -> /~{DBANK3_WR}
- U23 pad 1: (no net) -> /MDA4
- U23 pad 10: (no net) -> GND
- U23 pad 11: (no net) -> /MMA4
- U23 pad 12: Net-(U23-Pad12) -> /MMA5
- U23 pad 13: Net-(U23-Pad13) -> /MMA6
- U23 pad 14: (no net) -> /MMA7
- U23 pad 2: (no net) -> /MDA5
- U23 pad 3: (no net) -> /~{DBANK4_WR}
- U23 pad 4: (no net) -> /~{MRAS}
- U23 pad 6: (no net) -> /MMA0
- U23 pad 7: (no net) -> /MMA1
- U23 pad 8: (no net) -> /MMA2
- U23 pad 9: (no net) -> /MMA3
- U24 pad 1: /MBA18 -> +5V
- U24 pad 10: /~{DBANK2_RD} -> /REGMAP2
- U24 pad 11: /~{DBANK1_RD} -> unconnected-(U24-~{Q2}-Pad11)
- U24 pad 12: /~{DBANK4_WR} -> /#CD2
- U24 pad 13: /~{DBANK3_WR} -> /#CD3
- U24 pad 14: /~{DBANK2_WR} -> unconnected-(U24-~{Q3}-Pad14)
- U24 pad 15: /~{DBANK1_WR} -> /REGMAP3
- U24 pad 2: /MBA19 -> /REGMAP0
- U24 pad 3: /~{WR} -> unconnected-(U24-~{Q0}-Pad3)
- U24 pad 4: /~{MREQ} -> /#CD0
- U24 pad 5: /~{MCAS} -> /#CD1
- U24 pad 6: +5V -> unconnected-(U24-~{Q1}-Pad6)
- U24 pad 7: /~{DBANK4_RD} -> /REGMAP1
- U24 pad 9: /~{DBANK3_RD} -> /WRREG
- U27 pad 1: unconnected-(U27-Pad1) -> /REGBNK3
- U27 pad 10: (no net) -> /MBA21
- U27 pad 11: (no net) -> /MBA22
- U27 pad 12: (no net) -> GND
- U27 pad 13: (no net) -> /MBA23
- U27 pad 14: (no net) -> /MBA24
- U27 pad 2: unconnected-(U27-Pad2) -> /REGBNK2
- U27 pad 3: unconnected-(U27-Pad3) -> /REGBNK1
- U27 pad 4: (no net) -> /REGBNK0
- U27 pad 5: (no net) -> Net-(U11-A3)
- U27 pad 6: (no net) -> Net-(U11-A2)
- U27 pad 7: (no net) -> Net-(U11-A1)
- U27 pad 8: (no net) -> Net-(U11-A0)
- U27 pad 9: (no net) -> /MBA20
- U4 pad 1: /~{RESET} -> Net-(RN1-R4)
- U4 pad 10: unconnected-(U4B-~{S}-Pad10) -> (no net)
- U4 pad 11: unconnected-(U4B-C-Pad11) -> /#CA1
- U4 pad 12: unconnected-(U4B-D-Pad12) -> GND
- U4 pad 13: unconnected-(U4B-~{R}-Pad13) -> /#CA15
- U4 pad 14: unconnected-(U4C-VCC-Pad14) -> /~{NMIGAT}
- U4 pad 2: /CD0 -> Net-(RN1-R3)
- U4 pad 3: /~{CSPROT} -> Net-(RN1-R2)
- U4 pad 4: +5V -> Net-(RN1-R1)
- U4 pad 5: /MPROTEN -> /~{#IOREQ}
- U4 pad 6: unconnected-(U4A-~{Q}-Pad6) -> /~{#MREQ}
- U4 pad 7: unconnected-(U4C-GND-Pad7) -> /~{#RD}
- U4 pad 8: unconnected-(U4B-~{Q}-Pad8) -> /~{#WR}
- U4 pad 9: unconnected-(U4B-Q-Pad9) -> /#CA0
- U5 pad 1: /~{MWR} -> GND
- U5 pad 10: (no net) -> GND
- U5 pad 11: /~{CSCONF} -> /#CA4
- U5 pad 12: /~{RD} -> Net-(JP1-Pin_6)
- U5 pad 13: Net-(U5-Pad13) -> /#CA5
- U5 pad 14: unconnected-(U5E-VCC-Pad14) -> Net-(JP1-Pin_8)
- U5 pad 2: /~{MREQ} -> GND
- U5 pad 3: /~{WR} -> Net-(RN2-R8)
- U5 pad 4: Net-(U23-Pad13) -> /~{#IOREQ}
- U5 pad 5: /~{MWR} -> Net-(RN2-R7)
- U5 pad 6: /~{CURPROT} -> /#CA2
- U5 pad 7: unconnected-(U5E-GND-Pad7) -> Net-(JP1-Pin_2)
- U5 pad 8: (no net) -> /#CA3
- U5 pad 9: (no net) -> Net-(JP1-Pin_4)
- U6 pad 1: unconnected-(U6-G-Pad1) -> /~{#WR}
- U6 pad 11: /CA4 -> /MDA7
- U6 pad 12: unconnected-(U6-R4-Pad12) -> /MDA6
- U6 pad 13: /CA5 -> /MDA5
- U6 pad 14: unconnected-(U6-R5-Pad14) -> /MDA4
- U6 pad 15: /CA6 -> /MDA3
- U6 pad 16: unconnected-(U6-R6-Pad16) -> /MDA2
- U6 pad 17: /CA7 -> /MDA1
- U6 pad 18: unconnected-(U6-R7-Pad18) -> /MDA0
- U6 pad 19: /~{CARDSEL} -> /~{DRAMREQ}
- U6 pad 2: GND -> /#CD0
- U6 pad 3: unconnected-(U6-R0-Pad3) -> /#CD1
- U6 pad 4: /~{IOREQ} -> /#CD2
- U6 pad 5: unconnected-(U6-R1-Pad5) -> /#CD3
- U6 pad 6: /CA2 -> /#CD4
- U6 pad 7: unconnected-(U6-R2-Pad7) -> /#CD5
- U6 pad 8: /CA3 -> /#CD6
- U6 pad 9: unconnected-(U6-R3-Pad9) -> /#CD7
- U7 pad 1: Net-(U5-Pad13) -> GND
- U7 pad 10: unconnected-(U7-Pad10) -> GND
- U7 pad 11: unconnected-(U7-Pad11) -> /WRPROT
- U7 pad 12: unconnected-(U7-Pad12) -> /REGBNK4
- U7 pad 13: unconnected-(U7-Pad13) -> /#CD4
- U7 pad 14: unconnected-(U7E-VCC-Pad14) -> /#CD5
- U7 pad 2: /JENA19 -> /REGBNK0
- U7 pad 3: /CD0 -> /#CD0
- U7 pad 4: Net-(U23-Pad12) -> /#CD1
- U7 pad 5: GND -> /REGBNK1
- U7 pad 6: /~{NMI} -> /REGBNK2
- U7 pad 7: unconnected-(U7E-GND-Pad7) -> /#CD2
- U7 pad 8: unconnected-(U7-Pad8) -> /#CD3
- U7 pad 9: unconnected-(U7-Pad9) -> /REGBNK3
- U8 pad 1: /~{CARDSEL} -> /~{CSMAP}
- U8 pad 10: /~{WRMAP} -> /#CA14
- U8 pad 11: unconnected-(U8B-O1-Pad11) -> /REGMAP2
- U8 pad 12: /~{WRREG} -> Net-(U11-A3)
- U8 pad 13: /~{CSREG} -> /#CA15
- U8 pad 14: /~{CSMAP} -> /REGMAP3
- U8 pad 15: /~{WR} -> GND
- U8 pad 2: /CA1 -> /REGMAP0
- U8 pad 3: /CA0 -> /#CA12
- U8 pad 4: /~{CSMAP} -> Net-(U11-A0)
- U8 pad 5: /~{CSREG} -> /REGMAP1
- U8 pad 6: /~{CSPROT} -> /#CA13
- U8 pad 7: /~{CSCONF} -> Net-(U11-A1)
- U8 pad 9: unconnected-(U8B-O3-Pad9) -> Net-(U11-A2)
- U9 pad 1: GND -> +5V
- U9 pad 10: GND -> /MDA2
- U9 pad 11: /~{WRREG} -> /MMA4
- U9 pad 12: /REGBNK0 -> /MMA5
- U9 pad 13: /CD4 -> /MDA3
- U9 pad 14: /CD5 -> /MMA6
- U9 pad 15: /REGBNK1 -> /MMA7
- U9 pad 16: /REGBNK2 -> /MDA4
- U9 pad 17: /CD6 -> /MMA8
- U9 pad 18: /CD7 -> /MMA9
- U9 pad 19: /REGBNK3 -> /MMA10
- U9 pad 2: /REGMAP0 -> /~{MCAS0}
- U9 pad 20: +5V -> /MDA5
- U9 pad 3: /CD0 -> /MDA0
- U9 pad 4: /CD1 -> /MMA0
- U9 pad 5: /REGMAP1 -> /MMA1
- U9 pad 6: /REGMAP2 -> /MDA1
- U9 pad 7: /CD2 -> /MMA2
- U9 pad 8: /CD3 -> /MMA3
- U9 pad 9: /REGMAP3 -> GND
- X1 pad 8: Net-(U19-RCLK) -> Net-(U9-I1/CLK)
